File: schematics/cpu5/decoder.kicad_sch (KiCad schematic)
At the start: 52 parts, among them J1 Conn_01x12, J2 Conn_01x03, J3 Conn_01x40, J4 Conn_01x05, U1 74LS161, U10 74LS574, U11 74LS574, U12 74LS08, U13 74LS138, U14 74LS138, U15 74LS138, U16 74LS138, U17 74LS138, U18 74LS138, U19 74LS138, U2 74LS161, U20 74LS138, U21 74LS08, U22 74LS04, U23 74LS86, U24 74LS32, U25 74LS86, U26 74LS08, U27 74LS138, U28 74LS04, U29 74LS32, U30 74LS32, U31 74LS08, U32 74LS32, U33 74LS32, U34 74LS74, U35 74LS541, U36 74LS541, U4 74LS04, U42 74LS541, U5 74LS08, U6 74LS32, U7 74LS08, U8 74LS32, U82 74LS541, U9 74LS32

Commit message: verilator works, loop program works
Parts:
- removed INTERNAL_ADDRESS_CONN1: Conn_01x16, Connector_PinHeader_2.54mm:PinHeader_1x16_P2.54mm_Vertical, symbol Connector_Generic:Conn_01x16
- removed INTERNAL_DATA_CONN1, INTERNAL_DATA_CONN2, MEM_CTL1: Conn_01x08, Connector_PinHeader_2.54mm:PinHeader_1x08_P2.54mm_Vertical, symbol Connector_Generic:Conn_01x08
- removed J4: Conn_01x05, Connector_PinHeader_2.54mm:PinHeader_1x05_P2.54mm_Vertical, symbol Connector_Generic:Conn_01x05
- removed U82: 74LS541, Package_DIP:DIP-20_W7.62mm, symbol 7400_ice:74LS541
Connections:
- net iDATA0 is gone; now on net DATA0: CONN_DATA1.1 (Pin_1)
- net iDATA1 is gone; now on net DATA1: CONN_DATA1.2 (Pin_2)
- net iDATA2 is gone; now on net DATA2: CONN_DATA1.3 (Pin_3)
- net iDATA3 is gone; now on net DATA3: CONN_DATA1.4 (Pin_4)
- net iDATA4 is gone; now on net DATA4: CONN_DATA1.5 (Pin_5)
- net iDATA5 is gone; now on net DATA5: CONN_DATA1.6 (Pin_6)
- net iDATA6 is gone; now on net DATA6: CONN_DATA1.7 (Pin_7)
- net iDATA7 is gone; now on net DATA7: CONN_DATA1.8 (Pin_8)
- net RESET_bar: no longer names the net of U26.12 (A4), U28.4 (Y1)
Other:
- removed sheet Memory
- removed sheet Registers
- removed sheet alu
- moved on the sheet: JFlags1
