File: schematics/cpu5/alu.kicad_sch (KiCad schematic)
At the start: 22 parts, among them U71 74LS541, U72 74LS541, U73 74LS541, U74 74LS541, U75 74LS541, U76 74LS08, U77 74LS32, U78 74LS541, U79 74LS04, U80 74LS08, U81 74LS541

Commit message: os + ints work, ZF issue
Connections:
- net +5V: now also U80.2 (B1)
- net at U80.1 (A1): now also U76.8 (Y3)
- net at U80.3 (Y1): now also U75.3 (A1)
Other:
- moved on the sheet: U75, U76C, U77D, U80A

Commit message: flags ok
Parts:
- added U93: 74LS32, Package_DIP:DIP-14_W7.62mm, symbol 7400_ice:74LS32
Connections:
- net +5V: now also U93.14 (VCC); no longer U80.2 (B1)
- net F_Z: now also U93.5 (B2)
- net GND: now also U93.7 (GND)
- net aluop0: now also U79.13 (A5)
- net at U79.12 (Y5): now also U93.4 (A2)
- new net: U80.2 (B1), U93.6 (Y2)
Other:
- moved on the sheet: U79F
Changed lines of the file:
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@@
   (junction (at 154.94 69.85) (diameter 0) (color 0 0 0 0)
   )
+  (junction (at 515.62 41.91) (diameter 0) (color 0 0 0 0)
+  )
   (junction (at 538.48 41.91) (diameter 0) (color 0 0 0 0)
   )
@@
   (junction (at 96.52 231.14) (diameter 0) (color 0 0 0 0)
   )
+  (junction (at 515.62 16.51) (diameter 0) (color 0 0 0 0)
+  )
   (junction (at 59.69 66.04) (diameter 0) (color 0 0 0 0)
   )
@@
     (stroke (width 0) (type default) (color 0 0 0 0))
   )
+  (wire (pts (xy 196.85 208.28) (xy 199.39 208.28))
+    (stroke (width 0) (type default) (color 0 0 0 0))
+  )
   (wire (pts (xy 43.18 142.24) (xy 43.18 139.7))
     (stroke (width 0) (type default) (color 0 0 0 0))
@@
     (stroke (width 0) (type default) (color 0 0 0 0))
   )
-  (wire (pts (xy 199.39 213.36) (xy 199.39 215.9))
+  (wire (pts (xy 199.39 208.28) (xy 199.39 215.9))
     (stroke (width 0) (type default) (color 0 0 0 0))
   )
@@
     (stroke (width 0) (type default) (color 0 0 0 0))
   )
+  (wire (pts (xy 180.34 205.74) (xy 181.61 205.74))
+    (stroke (width 0) (type default) (color 0 0 0 0))
+  )
   (wire (pts (xy 48.26 181.61) (xy 48.26 193.04))
     (stroke (width 0) (type default) (color 0 0 0 0))
@@
     (stroke (width 0) (type default) (color 0 0 0 0))
   )
+  (wire (pts (xy 163.83 205.74) (xy 165.1 205.74))
+    (stroke (width 0) (type default) (color 0 0 0 0))
+  )
   (wire (pts (xy 233.68 83.82) (xy 236.22 83.82))
     (stroke (width 0) (type default) (color 0 0 0 0))
@@
     (stroke (width 0) (type default) (color 0 0 0 0))
   )
+  (wire (pts (xy 505.46 16.51) (xy 515.62 16.51))
+    (stroke (width 0) (type default) (color 0 0 0 0))
+  )
   (wire (pts (xy 46.99 31.75) (xy 46.99 34.29))
     (stroke (width 0) (type default) (color 0 0 0 0))
@@
     (stroke (width 0) (type default) (color 0 0 0 0))
   )
+  (wire (pts (xy 505.46 41.91) (xy 515.62 41.91))
+    (stroke (width 0) (type default) (color 0 0 0 0))
+  )
   (wire (pts (xy 133.35 127) (xy 111.76 127))
     (stroke (width 0) (type default) (color 0 0 0 0))
@@
     (stroke (width 0) (type default) (color 0 0 0 0))
   )
+  (wire (pts (xy 163.83 210.82) (xy 181.61 210.82))
+    (stroke (width 0) (type default) (color 0 0 0 0))
+  )
   (wire (pts (xy 129.54 243.84) (xy 129.54 246.38))
     (stroke (width 0) (type default) (color 0 0 0 0))
@@
     )
   )
+  (global_label "F_Z" (shape input) (at 163.83 210.82 180) (fields_autoplaced)
+    (effects (font (size 1.27 1.27)) (justify right))
+    (property "Intersheet References" "${INTERSHEET_REFS}" (id 0) (at 158.1512 210.7406 0)
+      (effects (font (size 1.27 1.27)) (justify right) hide)
+    )
+  )
   (global_label "Fo" (shape input) (at 425.45 43.18 0) (fields_autoplaced)
     (effects (font (size 1.27 1.27)) (justify left))
@@
     )
   )
+  (global_label "aluop0" (shape input) (at 163.83 205.74 180) (fields_autoplaced)
+    (effects (font (size 1.27 1.27)) (justify right))
+    (property "Intersheet References" "${INTERSHEET_REFS}" (id 0) (at 154.9459 205.6606 0)
+      (effects (font (size 1.27 1.27)) (justify right) hide)
+    )
+  )
   (global_label "aluop1" (shape input) (at 143.51 160.02 180) (fields_autoplaced)
     (effects (font (size 1.27 1.27)) (justify right))
@@
     (pin "1")
   )
-  (symbol (lib_id "power:+5V") (at 199.39 213.36 0) (unit 1)
+  (symbol (lib_id "7400_ice:74LS32") (at 429.26 180.34 0) (unit 4)
     (in_bom yes) (on_board yes) (fields_autoplaced)
-    (property "Reference" "#PWR?" (id 0) (at 199.39 217.17 0)
+    (property "Reference" "U93" (id 0) (at 429.26 171.45 0))
+    (property "Value" "74LS32" (id 1) (at 429.26 173.99 0))
+    (property "Footprint" "Package_DIP:DIP-14_W7.62mm" (id 2) (at 429.26 180.34 0)
       (effects (font (size 1.27 1.27)) hide)
     )
-    (property "Value" "+5V" (id 1) (at 199.39 208.28 0))
-    (property "Footprint" "" (id 2) (at 199.39 213.36 0)
+    (property "Datasheet" "http://www.ti.com/lit/gpn/sn74LS32" (id 3) (at 429.26 184.15 0)
       (effects (font (size 1.27 1.27)) hide)
     )
-    (property "Datasheet" "" (id 3) (at 199.39 213.36 0)
+    (property "VerilogInclude" "icechips/7432.v" (id 4) (at 429.26 180.34 0)
       (effects (font (size 1.27 1.27)) hide)
     )
-    (pin "1")
+    (property "VerilogCode" "ttl_7432 core (.A_2D({B4,A4,B3,A3,B2,A2,B1,A1}), .Y({Y4,Y3,Y2,Y1}));" (id 5) (at 429.26 180.34 0)
+      (effects (font (size 1.27 1.27)) hide)
+    )
+    (pin "11")
+    (pin "12")
+    (pin "13")
   )
   (symbol (lib_id "power:GND") (at 125.73 133.35 0) (unit 1)
@@
     (pin "1")
   )
-  (symbol (lib_id "7400_ice:74LS04") (at 471.17 177.8 0) (unit 6)
+  (symbol (lib_id "7400_ice:74LS04") (at 172.72 205.74 0) (unit 6)
     (in_bom yes) (on_board yes) (fields_autoplaced)
-    (property "Reference" "U79" (id 0) (at 471.17 163.83 0))
-    (property "Value" "74LS04" (id 1) (at 471.17 166.37 0))
-    (property "Footprint" "Package_DIP:DIP-14_W7.62mm" (id 2) (at 471.17 177.8 0)
+    (property "Reference" "U79" (id 0) (at 172.72 191.77 0))
+    (property "Value" "74LS04" (id 1) (at 172.72 194.31 0))
+    (property "Footprint" "Package_DIP:DIP-14_W7.62mm" (id 2) (at 172.72 205.74 0)
       (effects (font (size 1.27 1.27)) hide)
     )
-    (property "Datasheet" "http://www.ti.com/lit/gpn/sn74LS04" (id 3) (at 469.9 182.88 0)
+    (property "Datasheet" "http://www.ti.com/lit/gpn/sn74LS04" (id 3) (at 171.45 210.82 0)
       (effects (font (size 1.27 1.27)) hide)
     )
-    (property "VerilogInclude" "icechips/7404.v" (id 4) (at 471.17 168.91 0))
-    (property "VerilogCode" "ttl_7404 core (.A(`A), .Y(`Y));" (id 5) (at 471.17 171.45 0))
+    (property "VerilogInclude" "icechips/7404.v" (id 4) (at 172.72 196.85 0))
+    (property "VerilogCode" "ttl_7404 core (.A(`A), .Y(`Y));" (id 5) (at 172.72 199.39 0))
     (pin "12")
     (pin "13")
@@
     (pin "1")
   )
+  (symbol (lib_id "7400_ice:74LS32") (at 189.23 208.28 0) (unit 2)
+    (in_bom yes) (on_board yes) (fields_autoplaced)
+    (property "Reference" "U93" (id 0) (at 189.23 199.39 0))
+    (property "Value" "74LS32" (id 1) (at 189.23 201.93 0))
+    (property "Footprint" "Package_DIP:DIP-14_W7.62mm" (id 2) (at 189.23 208.28 0)
+      (effects (font (size 1.27 1.27)) hide)
+    )
+    (property "Datasheet" "http://www.ti.com/lit/gpn/sn74LS32" (id 3) (at 189.23 212.09 0)
+      (effects (font (size 1.27 1.27)) hide)
+    )
+    (property "VerilogInclude" "icechips/7432.v" (id 4) (at 189.23 208.28 0)
+      (effects (font (size 1.27 1.27)) hide)
+    )
+    (property "VerilogCode" "ttl_7432 core (.A_2D({B4,A4,B3,A3,B2,A2,B1,A1}), .Y({Y4,Y3,Y2,Y1}));" (id 5) (at 189.23 208.28 0)
+      (effects (font (size 1.27 1.27)) hide)
+    )
+    (pin "4")
+    (pin "5")
+    (pin "6")
+  )
   (symbol (lib_id "7400_ice:74LS08") (at 201.93 223.52 270) (unit 1)
     (in_bom yes) (on_board yes) (fields_autoplaced)
@@
     (pin "3")
   )
+  (symbol (lib_id "7400_ice:74LS32") (at 505.46 29.21 0) (unit 5)
+    (in_bom yes) (on_board yes) (fields_autoplaced)
+    (property "Reference" "U93" (id 0) (at 511.81 27.9399 0)
+      (effects (font (size 1.27 1.27)) (justify left))
+    )
+    (property "Value" "74LS32" (id 1) (at 511.81 30.4799 0)
+      (effects (font (size 1.27 1.27)) (justify left))
+    )
+    (property "Footprint" "Package_DIP:DIP-14_W7.62mm" (id 2) (at 505.46 29.21 0)
+      (effects (font (size 1.27 1.27)) hide)
+    )
+    (property "Datasheet" "http://www.ti.com/lit/gpn/sn74LS32" (id 3) (at 505.46 33.02 0)
+      (effects (font (size 1.27 1.27)) hide)
+    )
+    (property "VerilogInclude" "icechips/7432.v" (id 4) (at 505.46 29.21 0)
+      (effects (font (size 1.27 1.27)) hide)
+    )
+    (property "VerilogCode" "ttl_7432 core (.A_2D({B4,A4,B3,A3,B2,A2,B1,A1}), .Y({Y4,Y3,Y2,Y1}));" (id 5) (at 505.46 29.21 0)
+      (effects (font (size 1.27 1.27)) hide)
+    )
+    (pin "14")
+    (pin "7")
+  )
   (symbol (lib_id "7400_ice:74LS08") (at 289.56 82.55 0) (unit 4)
     (in_bom yes) (on_board yes)
@@
     (pin "6")
   )
+  (symbol (lib_id "7400_ice:74LS32") (at 429.26 139.7 0) (unit 1)
+    (in_bom yes) (on_board yes) (fields_autoplaced)
+    (property "Reference" "U93" (id 0) (at 429.26 130.81 0))
+    (property "Value" "74LS32" (id 1) (at 429.26 133.35 0))
+    (property "Footprint" "Package_DIP:DIP-14_W7.62mm" (id 2) (at 429.26 139.7 0)
+      (effects (font (size 1.27 1.27)) hide)
+    )
+    (property "Datasheet" "http://www.ti.com/lit/gpn/sn74LS32" (id 3) (at 429.26 143.51 0)
+      (effects (font (size 1.27 1.27)) hide)
+    )
+    (property "VerilogInclude" "icechips/7432.v" (id 4) (at 429.26 139.7 0)
+      (effects (font (size 1.27 1.27)) hide)
+    )
+    (property "VerilogCode" "ttl_7432 core (.A_2D({B4,A4,B3,A3,B2,A2,B1,A1}), .Y({Y4,Y3,Y2,Y1}));" (id 5) (at 429.26 139.7 0)
+      (effects (font (size 1.27 1.27)) hide)
+    )
+    (pin "1")
+    (pin "2")
+    (pin "3")
+  )
   (symbol (lib_id "power:GND") (at 139.7 48.26 0) (unit 1)
     (in_bom yes) (on_board yes) (fields_autoplaced)
@@
     (pin "1")
   )
+  (symbol (lib_id "7400_ice:74LS32") (at 429.26 166.37 0) (unit 3)
+    (in_bom yes) (on_board yes) (fields_autoplaced)
+    (property "Reference" "U93" (id 0) (at 429.26 157.48 0))
+    (property "Value" "74LS32" (id 1) (at 429.26 160.02 0))
+    (property "Footprint" "Package_DIP:DIP-14_W7.62mm" (id 2) (at 429.26 166.37 0)
+      (effects (font (size 1.27 1.27)) hide)
+    )
+    (property "Datasheet" "http://www.ti.com/lit/gpn/sn74LS32" (id 3) (at 429.26 170.18 0)
+      (effects (font (size 1.27 1.27)) hide)
+    )
+    (property "VerilogInclude" "icechips/7432.v" (id 4) (at 429.26 166.37 0)
+      (effects (font (size 1.27 1.27)) hide)
+    )
+    (property "VerilogCode" "ttl_7432 core (.A_2D({B4,A4,B3,A3,B2,A2,B1,A1}), .Y({Y4,Y3,Y2,Y1}));" (id 5) (at 429.26 166.37 0)
+      (effects (font (size 1.27 1.27)) hide)
+    )
+    (pin "10")
+    (pin "8")
+    (pin "9")
+  )
   (symbol (lib_id "power:GND") (at 515.62 43.18 0) (unit 1)

Commit message: Multithread + paging!
Parts:
- AROM_HIGH1, AROM_LOW1: VerilogInclude icechips/roms.v -> icechips/memory.v
- CONN_DATA3: footprint Connector_PinHeader_2.54mm:PinHeader_1x08_P2.54mm_Vertical -> Connector_PinHeader_2.54mm:PinHeader_1x09_P2.54mm_Vertical
Changed lines of the file:
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@@
       (effects (font (size 1.27 1.27) italic) hide)
     )
-    (property "VerilogInclude" "icechips/roms.v" (id 4) (at 103.505 180.34 0))
+    (property "VerilogInclude" "icechips/memory.v" (id 4) (at 103.505 180.34 0))
     (property "VerilogCode" "at28c64_rom #(.ROM_INDEX(2)) U(.A(`A), .D(`D), .nCE(_CE), .nOE(_OE), .nWE(_WE));" (id 5) (at 123.19 170.18 0)
       (effects (font (size 1.27 1.27)) hide)
@@
     (property "Reference" "CONN_DATA3" (id 0) (at 417.83 24.13 0))
     (property "Value" "Conn_01x08" (id 1) (at 417.83 26.67 0))
-    (property "Footprint" "Connector_PinHeader_2.54mm:PinHeader_1x08_P2.54mm_Vertical" (id 2) (at 417.83 38.1 0)
+    (property "Footprint" "Connector_PinHeader_2.54mm:PinHeader_1x09_P2.54mm_Vertical" (id 2) (at 417.83 38.1 0)
       (effects (font (size 1.27 1.27)) hide)
     )
@@
       (effects (font (size 1.27 1.27) italic) hide)
     )
-    (property "VerilogInclude" "icechips/roms.v" (id 4) (at 177.165 180.34 0))
+    (property "VerilogInclude" "icechips/memory.v" (id 4) (at 177.165 180.34 0))
     (property "VerilogCode" "at28c64_rom #(.ROM_INDEX(3)) U(.A(`A), .D(`D), .nCE(_CE), .nOE(_OE), .nWE(_WE));" (id 5) (at 196.85 170.18 0)
       (effects (font (size 1.27 1.27)) hide)
