File: schematics/cpu5/registers.kicad_sch (KiCad schematic)
At the start: 29 parts, among them U3 74LS193, U37 74LS193, U38 74LS541, U39 74LS193, U40 74LS193, U41 74LS541, U43 74LS541, U44 74LS541, U45 74LS193, U46 74LS193, U47 74LS541, U48 74LS193, U49 74LS193, U50 74LS193, U51 74LS193, U52 74LS541, U53 74LS541, U54 74LS541, U55 74LS541, U56 74LS193, U57 74LS193, U58 74LS541, U59 74LS541, U60 74LS541

Commit message: verilator works, loop program works
Parts:
- added CONN_CTL_M1: Conn_01x08, Connector_PinHeader_2.54mm:PinHeader_1x08_P2.54mm_Vertical, symbol Connector_Generic:Conn_01x08
- added MH1, ML1, U62: 74LS574, Package_DIP:DIP-20_W7.62mm, symbol 7400_ice:74LS574
- added U61: 74LS32, Package_DIP:DIP-14_W7.62mm, symbol 7400_ice:74LS32
- added U63, U64, U69, U70: 74LS541, Package_DIP:DIP-20_W7.62mm, symbol 7400_ice:74LS541
- added U65, U66, U67, U68: 74LS83, Package_DIP:DIP-16_W7.62mm, symbol 7400_ice:74LS83
- CONN_DATA2: VerilogModulePort 1,2,3,4,5,6,7,8 -> (none)
Connections:
- net +5V: now also U45.4 (CPD), MH1.20 (VCC), ML1.20 (VCC), U61.14 (VCC), U62.20 (VCC), U63.20 (VCC), U64.20 (VCC), U65.5 (VCC), U66.5 (VCC), U67.5 (VCC), U68.5 (VCC), U69.20 (VCC), U70.20 (VCC)
- net ADDR0: now also U69.18 (Y0)
- net ADDR1: now also U69.17 (Y1)
- net ADDR10: now also U70.16 (Y2)
- net ADDR11: now also U70.15 (Y3)
- net ADDR12: now also U70.14 (Y4)
- net ADDR13: now also U70.13 (Y5)
- net ADDR14: now also U70.12 (Y6)
- net ADDR15: now also U70.11 (Y7)
- net ADDR2: now also U69.16 (Y2)
- net ADDR3: now also U69.15 (Y3)
- net ADDR4: now also U69.14 (Y4)
- net ADDR5: now also U69.13 (Y5)
- net ADDR6: now also U69.12 (Y6)
- net ADDR7: now also U69.11 (Y7)
- net ADDR8: now also U70.18 (Y0)
- net ADDR9: now also U70.17 (Y1)
- net DATA0: now also MH1.2 (D0), ML1.2 (D0), U62.2 (D0), U63.18 (Y0), U64.18 (Y0)
- net DATA1: now also MH1.3 (D1), ML1.3 (D1), U62.3 (D1), U63.17 (Y1), U64.17 (Y1)
- net DATA2: now also MH1.4 (D2), ML1.4 (D2), U62.4 (D2), U63.16 (Y2), U64.16 (Y2)
- net DATA3: now also MH1.5 (D3), ML1.5 (D3), U62.5 (D3), U63.15 (Y3), U64.15 (Y3)
- net DATA4: now also MH1.6 (D4), ML1.6 (D4), U62.6 (D4), U63.14 (Y4), U64.14 (Y4)
- net DATA5: now also MH1.7 (D5), ML1.7 (D5), U62.7 (D5), U63.13 (Y5), U64.13 (Y5)
- net DATA6: now also MH1.8 (D6), ML1.8 (D6), U62.8 (D6), U63.12 (Y6), U64.12 (Y6)
- net DATA7: now also MH1.9 (D7), ML1.9 (D7), U62.9 (D7), U63.11 (Y7), U64.11 (Y7)
- net GND: now also MH1.1 (OE_bar), MH1.10 (GND), ML1.1 (OE_bar), ML1.10 (GND), U61.7 (GND), U62.1 (OE_bar), U62.10 (GND), U63.10 (GND), U63.19 (OE2_bar), U64.10 (GND), U64.19 (OE2_bar), U65.12 (GND), U65.13 (C0), U66.12 (GND), U67.12 (GND), U68.12 (GND), U69.10 (GND), U69.19 (OE2_bar), U70.10 (GND), U70.19 (OE2_bar); no longer U45.4 (CPD)
- new net: U61.2 (B1), U65.9 (S1)
- new net: U61.3 (Y1), U69.2 (A0)
- new net: U65.6 (S2), U69.3 (A1)
- new net: U65.2 (S3), U69.4 (A2)
- new net: U65.15 (S4), U69.5 (A3)
- new net: U66.9 (S1), U69.6 (A4)
- new net: U66.6 (S2), U69.7 (A5)
- new net: U66.2 (S3), U69.8 (A6)
- new net: U66.15 (S4), U69.9 (A7)
- new net: ML1.19 (Y0), U63.2 (A0), U65.10 (A1)
- new net: ML1.18 (Y1), U63.3 (A1), U65.8 (A2)
- new net: ML1.17 (Y2), U63.4 (A2), U65.3 (A3)
- new net: ML1.16 (Y3), U63.5 (A3), U65.1 (A4)
- new net: ML1.15 (Y4), U63.6 (A4), U66.10 (A1)
- new net: ML1.14 (Y5), U63.7 (A5), U66.8 (A2)
- new net: ML1.13 (Y6), U63.8 (A6), U66.3 (A3)
- new net: ML1.12 (Y7), U63.9 (A7), U66.1 (A4)
- new net: MH1.12 (Y7), U64.9 (A7), U68.1 (A4)
- new net: MH1.13 (Y6), U64.8 (A6), U68.3 (A3)
- new net: MH1.14 (Y5), U64.7 (A5), U68.8 (A2)
- new net: MH1.15 (Y4), U64.6 (A4), U68.10 (A1)
- new net: MH1.16 (Y3), U64.5 (A3), U67.1 (A4)
- new net: MH1.17 (Y2), U64.4 (A2), U67.3 (A3)
- new net: MH1.18 (Y1), U64.3 (A1), U67.8 (A2)
- new net: MH1.19 (Y0), U64.2 (A0), U67.10 (A1)
- new net: U62.15 (Y4), U66.11 (B1)
- new net: U65.14 (C4), U66.13 (C0)
- new net: U66.14 (C4), U67.13 (C0)
- new net: U62.12 (Y7), U66.16 (B4), U67.11 (B1), U67.16 (B4), U67.4 (B3), U67.7 (B2), U68.11 (B1), U68.16 (B4), U68.4 (B3), U68.7 (B2)
- new net: U62.13 (Y6), U66.4 (B3)
- new net: U62.14 (Y5), U66.7 (B2)
- new net: U67.14 (C4), U68.13 (C0)
- new net: U68.15 (S4), U70.9 (A7)
- new net: U68.2 (S3), U70.8 (A6)
- new net: U68.6 (S2), U70.7 (A5)
- new net: U68.9 (S1), U70.6 (A4)
- new net: U62.19 (Y0), U65.11 (B1)
- new net: U62.16 (Y3), U65.16 (B4)
- new net: U62.17 (Y2), U65.4 (B3)
- new net: U62.18 (Y1), U65.7 (B2)
- new net: U67.15 (S4), U70.5 (A3)
- new net: U67.2 (S3), U70.4 (A2)
- new net: U67.6 (S2), U70.3 (A1)
- new net: U67.9 (S1), U70.2 (A0)
- new net MFa: CONN_CTL_M1.7 (Pin_7), U69.1 (OE1_bar), U70.1 (OE1_bar)
- new net MHi: CONN_CTL_M1.6 (Pin_6), MH1.11 (CLK)
- new net MHo: CONN_CTL_M1.3 (Pin_3), U64.1 (OE1_bar)
- new net MLi: CONN_CTL_M1.5 (Pin_5), ML1.11 (CLK)
- new net MLo: CONN_CTL_M1.4 (Pin_4), U63.1 (OE1_bar)
- new net OFFi: CONN_CTL_M1.1 (Pin_1), U62.11 (CLK)
- new net SELhigh: CONN_CTL_M1.2 (Pin_2), U61.1 (A1)
Other:
- moved on the sheet: CONN_ADDRESS2, CONN_CTL_pB1, CONN_DATA2, U45, U46, U47, U49, U51, U53, U54, U55

Commit message: Multithread + paging!
Parts:
- U48, U49, U50, U51, U56, U57: footprint Package_DIP:DIP-8-16_W7.62mm -> Package_DIP:DIP-16_W7.62mm
Changed lines of the file:
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@@
     (property "Reference" "U50" (id 0) (at 435.61 54.3812 90))
     (property "Value" "74LS193" (id 1) (at 435.61 56.9212 90))
-    (property "Footprint" "Package_DIP:DIP-8-16_W7.62mm" (id 2) (at 417.83 60.96 0)
+    (property "Footprint" "Package_DIP:DIP-16_W7.62mm" (id 2) (at 417.83 60.96 0)
       (effects (font (size 1.27 1.27)) hide)
     )
@@
     (property "Reference" "U56" (id 0) (at 482.6 54.3812 90))
     (property "Value" "74LS193" (id 1) (at 482.6 56.9212 90))
-    (property "Footprint" "Package_DIP:DIP-8-16_W7.62mm" (id 2) (at 464.82 60.96 0)
+    (property "Footprint" "Package_DIP:DIP-16_W7.62mm" (id 2) (at 464.82 60.96 0)
       (effects (font (size 1.27 1.27)) hide)
     )
@@
     (property "Reference" "U49" (id 0) (at 524.51 299.4912 90))
     (property "Value" "74LS193" (id 1) (at 524.51 302.0312 90))
-    (property "Footprint" "Package_DIP:DIP-8-16_W7.62mm" (id 2) (at 506.73 306.07 0)
+    (property "Footprint" "Package_DIP:DIP-16_W7.62mm" (id 2) (at 506.73 306.07 0)
       (effects (font (size 1.27 1.27)) hide)
     )
@@
     (property "Reference" "U51" (id 0) (at 566.42 299.4912 90))
     (property "Value" "74LS193" (id 1) (at 566.42 302.0312 90))
-    (property "Footprint" "Package_DIP:DIP-8-16_W7.62mm" (id 2) (at 548.64 306.07 0)
+    (property "Footprint" "Package_DIP:DIP-16_W7.62mm" (id 2) (at 548.64 306.07 0)
       (effects (font (size 1.27 1.27)) hide)
     )
@@
     (property "Reference" "U48" (id 0) (at 393.7 54.3812 90))
     (property "Value" "74LS193" (id 1) (at 393.7 56.9212 90))
-    (property "Footprint" "Package_DIP:DIP-8-16_W7.62mm" (id 2) (at 375.92 60.96 0)
+    (property "Footprint" "Package_DIP:DIP-16_W7.62mm" (id 2) (at 375.92 60.96 0)
       (effects (font (size 1.27 1.27)) hide)
     )
@@
     (property "Reference" "U57" (id 0) (at 524.51 54.3812 90))
     (property "Value" "74LS193" (id 1) (at 524.51 56.9212 90))
-    (property "Footprint" "Package_DIP:DIP-8-16_W7.62mm" (id 2) (at 506.73 60.96 0)
-      (effects (font (size 1.27 1.27)) hide)
-    )
+    (property "Footprint" "Package_DIP:DIP-16_W7.62mm" (id 2) (at 506.73 60.96 0)
+      (effects (font (size 1.27 1.27)) hide)
+    )

Commit message: Page faults work
Parts:
- added IR_BUF3: 74LS574, Package_DIP:DIP-20_W7.62mm, symbol 7400_ice:74LS574
- added U136: 74LS541, Package_DIP:DIP-20_W7.62mm, symbol 7400_ice:74LS541
Connections:
- net +5V: now also IR_BUF3.20 (VCC), U136.20 (VCC)
- net DATA0: now also U136.2 (A0); no longer U62.2 (D0)
- net DATA1: now also U136.3 (A1); no longer U62.3 (D1)
- net DATA2: now also U136.4 (A2); no longer U62.4 (D2)
- net DATA3: now also U136.5 (A3); no longer U62.5 (D3)
- net DATA4: now also U136.6 (A4); no longer U62.6 (D4)
- net DATA5: now also U136.7 (A5); no longer U62.7 (D5)
- net DATA6: now also U136.8 (A6); no longer U62.8 (D6)
- net DATA7: now also U136.9 (A7); no longer U62.9 (D7)
- net GND: now also IR_BUF3.10 (GND), U136.10 (GND), U136.19 (OE2_bar)
- net at U62.15 (Y4), U66.11 (B1): now also IR_BUF3.6 (D4)
- net at U62.12 (Y7), U66.16 (B4), U67.11 (B1)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: now also IR_BUF3.9 (D7)
- net at U62.13 (Y6), U66.4 (B3): now also IR_BUF3.8 (D6)
- net at U62.14 (Y5), U66.7 (B2): now also IR_BUF3.7 (D5)
- net at U62.19 (Y0), U65.11 (B1): now also IR_BUF3.2 (D0)
- net at U62.16 (Y3), U65.16 (B4): now also IR_BUF3.5 (D3)
- net at U62.17 (Y2), U65.4 (B3): now also IR_BUF3.4 (D2)
- net at U62.18 (Y1), U65.7 (B2): now also IR_BUF3.3 (D1)
- new net: IR_BUF3.12 (Y7), U136.11 (Y7), U62.9 (D7)
- new net: IR_BUF3.13 (Y6), U136.12 (Y6), U62.8 (D6)
- new net: IR_BUF3.14 (Y5), U136.13 (Y5), U62.7 (D5)
- new net: IR_BUF3.15 (Y4), U136.14 (Y4), U62.6 (D4)
- new net: IR_BUF3.16 (Y3), U136.15 (Y3), U62.5 (D3)
- new net: IR_BUF3.17 (Y2), U136.16 (Y2), U62.4 (D2)
- new net: IR_BUF3.18 (Y1), U136.17 (Y1), U62.3 (D1)
- new net: IR_BUF3.19 (Y0), U136.18 (Y0), U62.2 (D0)
- new net LOAD_FAULT: U136.1 (OE1_bar)
- new net LOAD_FAULT_bar: IR_BUF3.1 (OE_bar)
- new net SAVE_FAULT: IR_BUF3.11 (CLK)
Other:
- moved on the sheet: U61E, U62
