File: schematics/cpu5/cpu5.kicad_pcb (KiCad board)
At the start: 2 copper layers, 45 parts, among them J1 Conn_01x12, J2 Conn_01x03, J3 Conn_01x40, U1 74LS161, U10 74LS574, U11 74LS574, U12 74LS08, U13 74LS138, U14 74LS138, U15 74LS138, U16 74LS138, U17 74LS138, U18 74LS138, U19 74LS138, U2 74LS161, U20 74LS138, U21 74LS08, U22 74LS04, U23 74LS86, U24 74LS32, U25 74LS86, U26 74LS08, U27 74LS138, U28 74LS04, U29 74LS32, U30 74LS32, U31 74LS08, U32 74LS32, U33 74LS32, U34 74LS74, U35 74LS541, U36 74LS541, U4 74LS04, U42 74LS541, U5 74LS08, U6 74LS32, U7 74LS08, U8 74LS32, U9 74LS32

Commit message: address marching with PC
Parts:
- added CONN_ADDRESS2: Conn_01x16, Connector_PinHeader_2.54mm:PinHeader_1x16_P2.54mm_Vertical, F.Cu at (132.0, 79.9)
- added CONN_CTL_S1: Conn_01x08, Connector_PinHeader_2.54mm:PinHeader_1x08_P2.54mm_Vertical, F.Cu at (190.9, 106.9)
- added CONN_CTL_pA1: Conn_01x08, Connector_PinHeader_2.54mm:PinHeader_1x08_P2.54mm_Vertical, F.Cu at (212.6, 79.9)
- added CONN_CTL_pB1: Conn_01x08, Connector_PinHeader_2.54mm:PinHeader_1x08_P2.54mm_Vertical, F.Cu at (186.3, 106.9)
- added CONN_DATA2: Conn_01x08, Connector_PinHeader_2.54mm:PinHeader_1x08_P2.54mm_Vertical, F.Cu at (217.3, 79.9)
- added JFlags1: Conn_01x04, Connector_PinHeader_1.00mm:PinHeader_1x04_P1.00mm_Vertical, F.Cu at (131.4, 157.3)
- added U3: 74LS193, Package_DIP:DIP-16_W7.62mm, F.Cu at (221.2, 79.7)
- added U37: 74LS193, Package_DIP:DIP-16_W7.62mm, F.Cu at (185.6, 129.1)
- added U38: 74LS541, Package_DIP:DIP-20_W7.62mm, F.Cu at (168.5, 79.7)
- added U39: 74LS193, Package_DIP:DIP-16_W7.62mm, F.Cu at (232.1, 79.7)
- added U40: 74LS193, Package_DIP:DIP-16_W7.62mm, F.Cu at (216.6, 102.1)
- added U41: 74LS541, Package_DIP:DIP-20_W7.62mm, F.Cu at (163.9, 106.7)
- added U43: 74LS541, Package_DIP:DIP-20_W7.62mm, F.Cu at (174.7, 106.7)
- added U44: 74LS541, Package_DIP:DIP-20_W7.62mm, F.Cu at (179.4, 79.7)
- added U45: 74LS193, Package_DIP:DIP-16_W7.62mm, F.Cu at (205.7, 106.7)
- added U46: 74LS193, Package_DIP:DIP-16_W7.62mm, F.Cu at (194.9, 106.7)
- added U47: 74LS541, Package_DIP:DIP-20_W7.62mm, F.Cu at (190.2, 79.7)
- added U48: 74LS193, Package_DIP:DIP-8-16_W7.62mm, F.Cu at (242.9, 79.7)
- added U49: 74LS193, Package_DIP:DIP-8-16_W7.62mm, F.Cu at (227.4, 101.5)
- added U50: 74LS193, Package_DIP:DIP-8-16_W7.62mm, F.Cu at (207.2, 128.6)
- added U51: 74LS193, Package_DIP:DIP-8-16_W7.62mm, F.Cu at (253.7, 79.7)
- added U52: 74LS541, Package_DIP:DIP-20_W7.62mm, F.Cu at (153.0, 106.7)
- added U53: 74LS541, Package_DIP:DIP-20_W7.62mm, F.Cu at (136.0, 79.7)
- added U54: 74LS541, Package_DIP:DIP-20_W7.62mm, F.Cu at (201.1, 79.7)
- added U55: 74LS541, Package_DIP:DIP-20_W7.62mm, F.Cu at (157.7, 79.7)
- added U56: 74LS193, Package_DIP:DIP-8-16_W7.62mm, F.Cu at (196.4, 128.6)
- added U57: 74LS193, Package_DIP:DIP-8-16_W7.62mm, F.Cu at (238.2, 101.5)
- added U58: 74LS541, Package_DIP:DIP-20_W7.62mm, F.Cu at (142.2, 106.7)
- added U59: 74LS541, Package_DIP:DIP-20_W7.62mm, F.Cu at (131.3, 122.4)
- added U60: 74LS541, Package_DIP:DIP-20_W7.62mm, F.Cu at (146.8, 79.7)
- moved U17 26.9 mm to (38.0, 82.8)
- moved U2 26.9 mm to (59.8, 82.8)
- moved U24 26.9 mm to (70.6, 82.8)
- moved U33 26.9 mm to (92.3, 92.6)
- moved U12 26.9 mm to (22.6, 127.5)
- moved U18 26.9 mm to (27.2, 82.8)
- moved CONN_ADDRESS1 26.9 mm to (27.9, 24.1)
- moved CONN_DATA1 26.9 mm to (89.5, 51.0)
- moved IR1 26.9 mm to (110.5, 23.8)
- moved J1 26.9 mm to (69.3, 24.1)
- moved J3 26.9 mm to (23.2, 24.1)
- moved Jdbg1 26.9 mm to (74.0, 24.1)
- moved U10 26.9 mm to (88.8, 23.8)
- moved U11 26.9 mm to (121.3, 23.8)
- moved U16 26.9 mm to (53.5, 61.0)
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Connections:
- net Net-(IR1-Pad2) renamed iIR0
- net Net-(IR1-Pad3) renamed iIR1
- net Net-(IR1-Pad4) renamed iIR2
- net Net-(IR1-Pad5) renamed iIR3
- net Net-(IR1-Pad6) renamed iIR4
- net Net-(IR1-Pad7) renamed iIR5
- net Net-(IR1-Pad8) renamed iIR6
- net Net-(IR1-Pad9) renamed iIR7
- CONN_DATA1 pad 2: DATA0 -> DATA1
- CONN_DATA1 pad 3: DATA0 -> DATA2
- CONN_DATA1 pad 4: DATA0 -> DATA3
- CONN_DATA1 pad 5: DATA0 -> DATA4
- CONN_DATA1 pad 6: DATA0 -> DATA5
- CONN_DATA1 pad 7: DATA0 -> DATA6
- CONN_DATA1 pad 8: DATA0 -> DATA7
- IR1 pad 1: DATA0 -> pACmm
- IR1 pad 10: DATA0 -> pACmm
- J1 pad 2: DATA0 -> pACmm
- MCODE_HIGH1 pad 14: DATA0 -> pACmm
- MCODE_HIGH1 pad 2: DATA0 -> pACmm
- MCODE_HIGH1 pad 20: DATA0 -> pACmm
- MCODE_HIGH1 pad 22: DATA0 -> pACmm
- MCODE_LOW1 pad 14: DATA0 -> pACmm
- MCODE_LOW1 pad 2: DATA0 -> pACmm
- MCODE_LOW1 pad 20: DATA0 -> pACmm
- MCODE_LOW1 pad 22: DATA0 -> pACmm
- U1 pad 3: DATA0 -> pACmm
- U1 pad 4: DATA0 -> pACmm
- U1 pad 5: DATA0 -> pACmm
- U1 pad 6: DATA0 -> pACmm
- U1 pad 8: DATA0 -> pACmm
- U1 pad 9: +5V -> Net-(U1-Pad9)
- U10 pad 1: DATA0 -> pACmm
- U10 pad 10: DATA0 -> pACmm
- U11 pad 1: DATA0 -> pACmm
- U11 pad 10: DATA0 -> pACmm
- U12 pad 7: DATA0 -> pACmm
- U13 pad 4: DATA0 -> pACmm
- U13 pad 8: DATA0 -> pACmm
- U14 pad 4: DATA0 -> pACmm
- U14 pad 8: DATA0 -> pACmm
- U15 pad 4: DATA0 -> pACmm
- U15 pad 8: DATA0 -> pACmm
- U16 pad 4: DATA0 -> pACmm
- U16 pad 8: DATA0 -> pACmm
- U17 pad 4: DATA0 -> pACmm
- U17 pad 8: DATA0 -> pACmm
- U18 pad 4: DATA0 -> pACmm
- U18 pad 8: DATA0 -> pACmm
- U19 pad 4: DATA0 -> pACmm
- U19 pad 8: DATA0 -> pACmm
- U2 pad 3: DATA0 -> pACmm
- U2 pad 4: DATA0 -> pACmm
- U2 pad 5: DATA0 -> pACmm
- U2 pad 6: DATA0 -> pACmm
- U2 pad 8: DATA0 -> pACmm
- U2 pad 9: +5V -> Net-(U1-Pad9)
- U20 pad 4: DATA0 -> pACmm
- U20 pad 8: DATA0 -> pACmm
- U21 pad 7: DATA0 -> pACmm
- U22 pad 7: DATA0 -> pACmm
- U23 pad 1: DATA0 -> F_SF
- U23 pad 10: DATA0 -> F_C
- U23 pad 2: DATA0 -> F_OF
- U23 pad 5: DATA0 -> F_Z
- U23 pad 7: DATA0 -> pACmm
- U24 pad 10: DATA0 -> F_C
- U24 pad 5: DATA0 -> F_Z
- U24 pad 7: DATA0 -> pACmm
- U24 pad 9: DATA0 -> F_Z
- U25 pad 7: DATA0 -> pACmm
- U26 pad 7: DATA0 -> pACmm
- U27 pad 4: DATA0 -> pACmm
- U27 pad 5: DATA0 -> pACmm
- U27 pad 8: DATA0 -> pACmm
- U28 pad 7: DATA0 -> pACmm
- U29 pad 7: DATA0 -> pACmm
- U30 pad 7: DATA0 -> pACmm
- U31 pad 7: DATA0 -> pACmm
- U32 pad 7: DATA0 -> pACmm
- U33 pad 7: DATA0 -> pACmm
- U34 pad 7: DATA0 -> pACmm
- U35 pad 1: DATA0 -> pACmm
- U35 pad 10: DATA0 -> pACmm
- U35 pad 7: DATA0 -> pACmm
- U36 pad 1: DATA0 -> pACmm
- U36 pad 10: DATA0 -> pACmm
- U36 pad 8: DATA0 -> pACmm
- U4 pad 12: unconnected-(U4-Pad12) -> Net-(U1-Pad9)
- U4 pad 7: DATA0 -> pACmm
- U42 pad 10: DATA0 -> pACmm
- U42 pad 19: DATA0 -> pACmm
- U5 pad 7: DATA0 -> pACmm
- U6 pad 7: DATA0 -> pACmm
- U7 pad 7: DATA0 -> pACmm
- U8 pad 10: DATA0 -> pACmm
- U8 pad 12: DATA0 -> DATA3
- U8 pad 13: DATA0 -> pACmm
- U8 pad 2: DATA0 -> pACmm
- U8 pad 4: DATA0 -> DATA1
- U8 pad 5: DATA0 -> pACmm
- U8 pad 7: DATA0 -> pACmm
- U8 pad 9: DATA0 -> DATA2
- U9 pad 1: DATA0 -> DATA4
- U9 pad 10: DATA0 -> pACmm
- U9 pad 12: DATA0 -> DATA7
- U9 pad 13: DATA0 -> pACmm
- U9 pad 2: DATA0 -> pACmm
- U9 pad 4: DATA0 -> DATA5
- U9 pad 5: DATA0 -> pACmm
- U9 pad 7: DATA0 -> pACmm
- U9 pad 9: DATA0 -> DATA6

Commit message: verilator works, loop program works
Parts:
- added ALU_DATA_BUS1: Conn_01x08, Connector_PinHeader_2.54mm:PinHeader_1x08_P2.54mm_Vertical, F.Cu at (221.0, 53.3)
- added ALU_OP_CONN1: Conn_01x05, Connector_PinHeader_2.54mm:PinHeader_1x05_P2.54mm_Vertical, F.Cu at (177.6, 99.7)
- added AROM_HIGH1: AT28C64-20PI, Package_DIP:DIP-28_W15.24mm, F.Cu at (158.4, 63.2)
- added AROM_LOW1: AT28C64-20PI, Package_DIP:DIP-28_W15.24mm, F.Cu at (158.4, 26.1)
- added CONN_CTL_M1: Conn_01x08, Connector_PinHeader_2.54mm:PinHeader_1x08_P2.54mm_Vertical, F.Cu at (33.6, 206.6)
- added CONN_DATA3: Conn_01x08, Connector_PinHeader_2.54mm:PinHeader_1x08_P2.54mm_Vertical, F.Cu at (225.6, 53.3)
- added INTERNAL_ADDRESS_CONN1: Conn_01x16, Connector_PinHeader_2.54mm:PinHeader_1x16_P2.54mm_Vertical, F.Cu at (125.3, 152.6)
- added INTERNAL_DATA_CONN1: Conn_01x08, Connector_PinHeader_2.54mm:PinHeader_1x08_P2.54mm_Vertical, F.Cu at (134.6, 152.6)
- added J4: Conn_01x05, Connector_PinHeader_2.54mm:PinHeader_1x05_P2.54mm_Vertical, F.Cu at (-8.27, 69.1)
- added JFlags2: Conn_01x04, Connector_PinHeader_1.00mm:PinHeader_1x04_P1.00mm_Vertical, F.Cu at (181.6, 98.9)
- added MEM_CTL1: Conn_01x08, Connector_PinHeader_2.54mm:PinHeader_1x08_P2.54mm_Vertical, F.Cu at (143.9, 152.6)
- added MH1: 74LS574, Package_DIP:DIP-20_W7.62mm, F.Cu at (45.3, 152.3)
- added ML1: 74LS574, Package_DIP:DIP-20_W7.62mm, F.Cu at (-13.6, 222.1)
- added ML2: 74LS574, Package_DIP:DIP-20_W7.62mm, F.Cu at (209.4, 53.1)
- added ML3: 74LS574, Package_DIP:DIP-20_W7.62mm, F.Cu at (187.7, 53.1)
- added ML4: 74LS574, Package_DIP:DIP-20_W7.62mm, F.Cu at (220.3, 26.1)
- added ML5: 74LS574, Package_DIP:DIP-20_W7.62mm, F.Cu at (198.6, 26.1)
- added ML6: 74LS574, Package_DIP:DIP-20_W7.62mm, F.Cu at (176.9, 53.1)
- added SIM_ADDRESS_CONN1: Conn_01x16, Connector_PinHeader_2.54mm:PinHeader_1x16_P2.54mm_Vertical, F.Cu at (125.3, 195.3)
- added SIM_DATA_CONN1: Conn_01x08, Connector_PinHeader_2.54mm:PinHeader_1x08_P2.54mm_Vertical, F.Cu at (139.3, 152.6)
- added SIM_MEM_CTL1: Conn_01x08, Connector_PinHeader_2.54mm:PinHeader_1x08_P2.54mm_Vertical, F.Cu at (130.0, 152.6)
- added U61: 74LS32, Package_DIP:DIP-14_W7.62mm, F.Cu at (-2.77, 233.3)
- added U62: 74LS574, Package_DIP:DIP-20_W7.62mm, F.Cu at (8.08, 206.3)
- added U63: 74LS541, Package_DIP:DIP-20_W7.62mm, F.Cu at (77.8, 152.3)
- added U64: 74LS541, Package_DIP:DIP-20_W7.62mm, F.Cu at (8.08, 179.3)
- added U65: 74LS83, Package_DIP:DIP-16_W7.62mm, F.Cu at (77.8, 179.3)
- added U66: 74LS83, Package_DIP:DIP-16_W7.62mm, F.Cu at (29.8, 228.7)
- added U67: 74LS83, Package_DIP:DIP-16_W7.62mm, F.Cu at (37.5, 206.3)
- added U68: 74LS83, Package_DIP:DIP-16_W7.62mm, F.Cu at (62.3, 201.7)
- added U69: 74LS541, Package_DIP:DIP-20_W7.62mm, F.Cu at (29.8, 179.3)
- added U70: 74LS541, Package_DIP:DIP-20_W7.62mm, F.Cu at (18.9, 179.3)
- added U71: 74LS541, Package_DIP:DIP-20_W7.62mm, F.Cu at (198.6, 53.1)
- added U72: 74LS541, Package_DIP:DIP-20_W7.62mm, F.Cu at (231.1, 26.1)
- added U73: 74LS541, Package_DIP:DIP-20_W7.62mm, F.Cu at (187.7, 26.1)
- added U74: 74LS541, Package_DIP:DIP-20_W7.62mm, F.Cu at (209.4, 26.1)
- added U75: 74LS541, Package_DIP:DIP-20_W7.62mm, F.Cu at (242.0, 26.1)
- added U76: 74LS08, Package_DIP:DIP-14_W7.62mm, F.Cu at (229.6, 53.1)
- added U77: 74LS32, Package_DIP:DIP-14_W7.62mm, F.Cu at (187.7, 80.1)
- added U78: 74LS541, Package_DIP:DIP-20_W7.62mm, F.Cu at (158.5, 100.4)
- added U79: 74LS04, Package_DIP:DIP-14_W7.62mm, F.Cu at (198.6, 80.1)
- added U80: 74LS08, Package_DIP:DIP-14_W7.62mm, F.Cu at (176.9, 80.1)
- added U81: 74LS541, Package_DIP:DIP-20_W7.62mm, F.Cu at (176.9, 26.1)
- moved U39 260.1 mm to (18.9, 228.7)
- moved CONN_DATA2 230.9 mm to (24.3, 206.6)
- moved U49 225.7 mm to (40.6, 228.2)
- moved U44 224.9 mm to (-13.6, 195.1)
- moved CONN_CTL_pA1 223.1 mm to (28.9, 206.6)
- moved U54 222.3 mm to (-8.97, 152.3)
- moved CONN_CTL_pB1 194.2 mm to (19.6, 206.6)
- moved U51 190.2 mm to (88.6, 174.2)
- moved U32 189.2 mm to (-13.6, 129.8)
- moved U57 183.6 mm to (83.9, 201.2)
- moved U43 178.8 mm to (1.88, 152.3)
- moved U50 175.9 mm to (59.2, 223.6)
- moved U52 171.9 mm to (-2.77, 179.3)
- moved U48 171.8 mm to (99.4, 174.2)
- moved U40 168.4 mm to (67.0, 179.3)
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Connections:
- net Net-(U48-Pad12) renamed pAdbg_TUD_bar
- net Net-(U48-Pad13) renamed pAdbg_TCD_bar
- net Net-(U48-Pad2) renamed pAdbg1
- net Net-(U48-Pad3) renamed pAdbg0
- net Net-(U48-Pad6) renamed pAdbg2
- net Net-(U48-Pad7) renamed pAdbg3
- net Net-(U50-Pad2) renamed pAdbg5
- net Net-(U50-Pad3) renamed pAdbg4
- net Net-(U50-Pad6) renamed pAdbg6
- net Net-(U50-Pad7) renamed pAdbg7
- CONN_CTL_pA1 pad 8: pArst -> RESET_bar
- CONN_CTL_pB1 pad 8: pBrst -> RESET_bar
- CONN_DATA1 pad 1: DATA0 -> iDATA0
- CONN_DATA1 pad 2: DATA1 -> iDATA1
- CONN_DATA1 pad 3: DATA2 -> iDATA2
- CONN_DATA1 pad 4: DATA3 -> iDATA3
- CONN_DATA1 pad 5: DATA4 -> iDATA4
- CONN_DATA1 pad 6: DATA5 -> iDATA5
- CONN_DATA1 pad 7: DATA6 -> iDATA6
- CONN_DATA1 pad 8: DATA7 -> iDATA7
- IR1 pad 1: pACmm -> GND
- IR1 pad 10: pACmm -> GND
- J1 pad 2: pACmm -> GND
- MCODE_HIGH1 pad 14: pACmm -> GND
- MCODE_HIGH1 pad 2: pACmm -> GND
- MCODE_HIGH1 pad 20: pACmm -> GND
- MCODE_HIGH1 pad 22: pACmm -> GND
- MCODE_LOW1 pad 14: pACmm -> GND
- MCODE_LOW1 pad 2: pACmm -> GND
- MCODE_LOW1 pad 20: pACmm -> GND
- MCODE_LOW1 pad 22: pACmm -> GND
- U1 pad 3: pACmm -> GND
- U1 pad 4: pACmm -> GND
- U1 pad 5: pACmm -> GND
- U1 pad 6: pACmm -> GND
- U1 pad 8: pACmm -> GND
- U10 pad 1: pACmm -> GND
- U10 pad 10: pACmm -> GND
- U11 pad 1: pACmm -> GND
- U11 pad 10: pACmm -> GND
- U12 pad 7: pACmm -> GND
- U13 pad 4: pACmm -> GND
- U13 pad 8: pACmm -> GND
- U14 pad 4: pACmm -> GND
- U14 pad 8: pACmm -> GND
- U15 pad 4: pACmm -> GND
- U15 pad 8: pACmm -> GND
- U16 pad 4: pACmm -> GND
- U16 pad 8: pACmm -> GND
- U17 pad 4: pACmm -> GND
- U17 pad 8: pACmm -> GND
- U18 pad 4: pACmm -> GND
- U18 pad 8: pACmm -> GND
- U19 pad 4: pACmm -> GND
- U19 pad 8: pACmm -> GND
- U2 pad 3: pACmm -> GND
- U2 pad 4: pACmm -> GND
- U2 pad 5: pACmm -> GND
- U2 pad 6: pACmm -> GND
- U2 pad 8: pACmm -> GND
- U20 pad 4: pACmm -> GND
- U20 pad 8: pACmm -> GND
- U21 pad 7: pACmm -> GND
- U22 pad 7: pACmm -> GND
- U23 pad 7: pACmm -> GND
- U24 pad 7: pACmm -> GND
- U25 pad 7: pACmm -> GND
- U26 pad 12: Net-(U26-Pad12) -> RESET_bar
- U26 pad 7: pACmm -> GND
- U27 pad 4: pACmm -> GND
- U27 pad 5: pACmm -> GND
- U27 pad 8: pACmm -> GND
- U28 pad 4: Net-(U26-Pad12) -> RESET_bar
- U28 pad 7: pACmm -> GND
- U29 pad 7: pACmm -> GND
- U3 pad 8: pACmm -> GND
- U30 pad 7: pACmm -> GND
- U31 pad 7: pACmm -> GND
- U32 pad 7: pACmm -> GND
- U33 pad 7: pACmm -> GND
- U34 pad 7: pACmm -> GND
- U35 pad 1: pACmm -> GND
- U35 pad 10: pACmm -> GND
- U35 pad 7: pACmm -> GND
- U36 pad 1: pACmm -> GND
- U36 pad 10: pACmm -> GND
- U36 pad 8: pACmm -> GND
- U37 pad 8: pACmm -> GND
- U38 pad 10: pACmm -> GND
- U38 pad 19: pACmm -> GND
- U39 pad 8: pACmm -> GND
- U4 pad 7: pACmm -> GND
- U40 pad 8: pACmm -> GND
- U41 pad 10: pACmm -> GND
- U41 pad 19: pACmm -> GND
- U42 pad 10: pACmm -> GND
- U42 pad 19: pACmm -> GND
- U43 pad 10: pACmm -> GND
- U43 pad 19: pACmm -> GND
- U44 pad 10: pACmm -> GND
- U44 pad 19: pACmm -> GND
- U45 pad 14: pBrst -> RESET_bar
- U45 pad 4: pACmm -> +5V
- U45 pad 8: pACmm -> GND
- U46 pad 14: pBrst -> RESET_bar
- U46 pad 8: pACmm -> GND
- U47 pad 10: pACmm -> GND
- U47 pad 19: pACmm -> GND
- U48 pad 4: pACmm -> +5V
- U48 pad 8: pACmm -> GND
- U49 pad 8: pACmm -> GND
- U5 pad 7: pACmm -> GND
- U50 pad 8: pACmm -> GND
- U51 pad 8: pACmm -> GND
- U52 pad 10: pACmm -> GND
- U52 pad 19: pACmm -> GND
- U53 pad 10: pACmm -> GND
- U53 pad 19: pACmm -> GND
- U54 pad 10: pACmm -> GND
- U54 pad 19: pACmm -> GND
- U55 pad 10: pACmm -> GND
- U55 pad 19: pACmm -> GND
- U56 pad 8: pACmm -> GND
- U57 pad 8: pACmm -> GND
- U58 pad 10: pACmm -> GND
- U58 pad 19: pACmm -> GND
- U59 pad 10: pACmm -> GND
- U59 pad 19: pACmm -> GND
- U6 pad 7: pACmm -> GND
- U60 pad 10: pACmm -> GND
- U60 pad 19: pACmm -> GND
- U7 pad 7: pACmm -> GND
- U8 pad 1: DATA0 -> iDATA0
- U8 pad 10: pACmm -> GND
- U8 pad 12: DATA3 -> iDATA3
- U8 pad 13: pACmm -> GND
- U8 pad 2: pACmm -> GND
- U8 pad 4: DATA1 -> iDATA1
- U8 pad 5: pACmm -> GND
- U8 pad 7: pACmm -> GND
- U8 pad 9: DATA2 -> iDATA2
- U9 pad 1: DATA4 -> iDATA4
- U9 pad 10: pACmm -> GND
- U9 pad 12: DATA7 -> iDATA7
- U9 pad 13: pACmm -> GND
- U9 pad 2: pACmm -> GND
- U9 pad 4: DATA5 -> iDATA5
- U9 pad 5: pACmm -> GND
- U9 pad 7: pACmm -> GND
- U9 pad 9: DATA6 -> iDATA6

Commit message: os + ints work, ZF issue
Parts:
- added DbgConn1: Conn_01x04, Connector_PinHeader_1.00mm:PinHeader_1x04_P1.00mm_Vertical, F.Cu at (307.3, 137.2)
- added DbgConn2: Conn_01x04, Connector_PinHeader_1.00mm:PinHeader_1x04_P1.00mm_Vertical, F.Cu at (315.0, 137.2)
- added INTERNAL_ADDRESS_CONN1: Conn_01x16, Connector_PinHeader_2.54mm:PinHeader_1x16_P2.54mm_Vertical, F.Cu at (171.8, 138.0)
- added INTERNAL_DATA_CONN1: Conn_01x08, Connector_PinHeader_2.54mm:PinHeader_1x08_P2.54mm_Vertical, F.Cu at (191.9, 138.0)
- added INTERNAL_DATA_CONN2: Conn_01x08, Connector_PinHeader_2.54mm:PinHeader_1x08_P2.54mm_Vertical, F.Cu at (196.6, 138.0)
- added INTERNAL_DATA_CONN3: Conn_01x08, Connector_PinHeader_2.54mm:PinHeader_1x08_P2.54mm_Vertical, F.Cu at (242.4, 138.0)
- added IRQ_conn1: Conn_01x04, Connector_PinHeader_1.00mm:PinHeader_1x04_P1.00mm_Vertical, F.Cu at (171.1, 179.9)
- added IntBoardConn1: Conn_01x04, Connector_PinHeader_1.00mm:PinHeader_1x04_P1.00mm_Vertical, F.Cu at (246.4, 137.2)
- added IntBoardConn2: Conn_01x04, Connector_PinHeader_1.00mm:PinHeader_1x04_P1.00mm_Vertical, F.Cu at (220.0, 164.2)
- added MEM_CTL1: Conn_01x08, Connector_PinHeader_2.54mm:PinHeader_1x08_P2.54mm_Vertical, F.Cu at (187.2, 138.0)
- added ML7: 74LS574, Package_DIP:DIP-20_W7.62mm, F.Cu at (220.0, 137.7)
- added U82: 74LS541, Package_DIP:DIP-20_W7.62mm, F.Cu at (175.7, 137.7)
- added U83: 74LS08, Package_DIP:DIP-14_W7.62mm, F.Cu at (296.4, 137.7)
- added U84: 74LS32, Package_DIP:DIP-14_W7.62mm, F.Cu at (285.6, 137.7)
- added U85: 74LS32, Package_DIP:DIP-14_W7.62mm, F.Cu at (253.0, 157.1)
- added U86: 74LS04, Package_DIP:DIP-14_W7.62mm, F.Cu at (253.0, 137.7)
- added U87: 74LS02, Package_DIP:DIP-14_W7.62mm, F.Cu at (309.9, 165.1)
- added U87: 74LS00, Package_DIP:DIP-14_W7.62mm, F.Cu at (274.7, 157.1)
- added U88: 74LS00, Package_DIP:DIP-14_W7.62mm, F.Cu at (263.9, 157.1)
- added U88: 74LS02, Package_DIP:DIP-14_W7.62mm, F.Cu at (320.7, 165.1)
- added U89: 74LS08, Package_DIP:DIP-14_W7.62mm, F.Cu at (263.9, 137.7)
- added U90: 74LS32, Package_DIP:DIP-14_W7.62mm, F.Cu at (285.6, 157.1)
- added U91: 74LS541, Package_DIP:DIP-20_W7.62mm, F.Cu at (230.8, 137.7)
- added U92: 74LS32, Package_DIP:DIP-14_W7.62mm, F.Cu at (274.7, 137.7)
Connections:
- U15 pad 10: ei -> Net-(U15-Pad10)
- U28 pad 1: unconnected-(U28-Pad1) -> Net-(U15-Pad10)
- U28 pad 2: unconnected-(U28-Pad2) -> ei
- U8 pad 1: iDATA0 -> DATA0
- U8 pad 10: GND -> IRQ
- U8 pad 12: iDATA3 -> DATA3
- U8 pad 13: GND -> IRQ
- U8 pad 2: GND -> IRQ
- U8 pad 4: iDATA1 -> DATA1
- U8 pad 5: GND -> IRQ
- U8 pad 9: iDATA2 -> DATA2
- U9 pad 1: iDATA4 -> DATA4
- U9 pad 10: GND -> IRQ
- U9 pad 12: iDATA7 -> DATA7
- U9 pad 13: GND -> IRQ
- U9 pad 2: GND -> IRQ
- U9 pad 4: iDATA5 -> DATA5
- U9 pad 5: GND -> IRQ
- U9 pad 9: iDATA6 -> DATA6

Commit message: Multithread + paging!
Parts:
- removed the INTERNAL_ADDRESS_CONN1 at (171.8, 138.0)
- removed the INTERNAL_ADDRESS_CONN1 at (125.3, 152.6)
- removed the INTERNAL_DATA_CONN1 at (134.6, 152.6)
- removed the INTERNAL_DATA_CONN1 at (191.9, 138.0)
- removed the MEM_CTL1 at (143.9, 152.6)
- removed the MEM_CTL1 at (187.2, 138.0)
- removed SIM_ADDRESS_CONN1: Conn_01x16, Connector_PinHeader_2.54mm:PinHeader_1x16_P2.54mm_Vertical
- removed SIM_DATA_CONN1, SIM_MEM_CTL1: Conn_01x08, Connector_PinHeader_2.54mm:PinHeader_1x08_P2.54mm_Vertical
- removed the U87 at (309.9, 165.1)
- removed the U87 at (274.7, 157.1)
- removed the U88 at (263.9, 157.1)
- removed the U88 at (320.7, 165.1)
- added INTERNAL_ADDRESS_CONN1: Conn_01x16, Connector_PinHeader_2.54mm:PinHeader_1x16_P2.54mm_Vertical, F.Cu at (-14.4, 24.6)
- added INTERNAL_ADDRESS_CONN2: Conn_01x16, Connector_PinHeader_2.54mm:PinHeader_1x16_P2.54mm_Vertical, F.Cu at (155.0, 24.6)
- added INTERNAL_DATA_CONN1: Conn_01x08, Connector_PinHeader_2.54mm:PinHeader_1x08_P2.54mm_Vertical, F.Cu at (-9.77, 61.7)
- added INTERNAL_DATA_CONN4: Conn_01x08, Connector_PinHeader_2.54mm:PinHeader_1x08_P2.54mm_Vertical, F.Cu at (155.0, 104.5)
- added INTERNAL_DATA_CONN5: Conn_01x08, Connector_PinHeader_2.54mm:PinHeader_1x08_P2.54mm_Vertical, F.Cu at (195.1, 61.7)
- added IntBoardConn3: Conn_01x04, Connector_PinHeader_1.00mm:PinHeader_1x04_P1.00mm_Vertical, F.Cu at (310.6, 43.2)
- added J5: Conn_01x03, Connector_PinHeader_2.54mm:PinHeader_1x03_P2.54mm_Vertical, F.Cu at (-14.4, 67.3)
- added MEM_CTL1: Conn_01x08, Connector_PinHeader_2.54mm:PinHeader_1x08_P2.54mm_Vertical, F.Cu at (-5.12, 61.7)
- added ML8: 74LS574, Package_DIP:DIP-20_W7.62mm, F.Cu at (199.0, 51.3)
- added U100: CY62256-70PC, Package_DIP:DIP-28_W15.24mm, F.Cu at (154.2, 67.1)
- added U101: 74LS04, Package_DIP:DIP-14_W7.62mm, F.Cu at (264.1, 24.3)
- added U102: 74LS02, Package_DIP:DIP-14_W7.62mm, F.Cu at (253.3, 43.7)
- added U103: 74LS541, Package_DIP:DIP-20_W7.62mm, F.Cu at (172.7, 88.5)
- added U104: 74LS541, Package_DIP:DIP-20_W7.62mm, F.Cu at (172.7, 61.5)
- added U105: 74LS541, Package_DIP:DIP-20_W7.62mm, F.Cu at (220.7, 51.3)
- added U106: 74LS541, Package_DIP:DIP-20_W7.62mm, F.Cu at (209.9, 51.3)
- added U107: 74LS541, Package_DIP:DIP-20_W7.62mm, F.Cu at (209.9, 24.3)
- added U108: 74LS02, Package_DIP:DIP-14_W7.62mm, F.Cu at (194.4, 103.3)
- added U109: 74LS32, Package_DIP:DIP-14_W7.62mm, F.Cu at (216.1, 78.3)
- added U110: AT28C64-20PI, Package_DIP:DIP-28_W7.62mm, F.Cu at (158.9, 24.3)
- added U111: AT28C64-20PI, Package_DIP:DIP-28_W7.62mm, F.Cu at (188.2, 24.3)
- added U112: 74LS32, Package_DIP:DIP-14_W7.62mm, F.Cu at (205.2, 78.3)
- added U113: 74LS32, Package_DIP:DIP-14_W7.62mm, F.Cu at (233.7, 81.3)
- added U114: 74LS138, Package_DIP:DIP-16_W7.62mm, F.Cu at (231.6, 51.3)
- added U115: 74LS541, Package_DIP:DIP-20_W7.62mm, F.Cu at (199.0, 24.3)
- added U116: 74LS541, Package_DIP:DIP-20_W7.62mm, F.Cu at (231.6, 24.3)
- added U117: 74LS138, Package_DIP:DIP-16_W7.62mm, F.Cu at (158.9, 104.2)
- added U118: 74LS541, Package_DIP:DIP-20_W7.62mm, F.Cu at (183.5, 61.5)
- added U119: 74LS541, Package_DIP:DIP-20_W7.62mm, F.Cu at (220.7, 24.3)
- added U87: 74LS02, Package_DIP:DIP-14_W7.62mm, F.Cu at (288.9, 46.7)
- added U88: 74LS02, Package_DIP:DIP-14_W7.62mm, F.Cu at (278.0, 97.7)
- added U93: 74LS32, Package_DIP:DIP-14_W7.62mm, F.Cu at (132.3, 204.6)
- added U94: 74LS541, Package_DIP:DIP-20_W7.62mm, F.Cu at (183.5, 88.5)
- added U95: 74LS32, Package_DIP:DIP-14_W7.62mm, F.Cu at (242.4, 46.2)
- added U96: 74LS138, Package_DIP:DIP-16_W7.62mm, F.Cu at (242.4, 24.3)
- added U97: 74LS00, Package_DIP:DIP-14_W7.62mm, F.Cu at (253.3, 24.3)
- added U98: 28C256, Package_DIP:DIP-28_W15.24mm, F.Cu at (169.7, 24.3)
- added U99: 74LS08, Package_DIP:DIP-14_W7.62mm, F.Cu at (194.4, 83.9)
- CONN_DATA3: footprint Connector_PinHeader_2.54mm:PinHeader_1x08_P2.54mm_Vertical -> Connector_PinHeader_2.54mm:PinHeader_1x09_P2.54mm_Vertical
- U48, U49, U50, U51, U56, U57: footprint Package_DIP:DIP-8-16_W7.62mm -> Package_DIP:DIP-16_W7.62mm
- moved DbgConn2 337.6 mm to (-19.7, 93.0)
- moved U75 236.5 mm to (113.9, 224.8)
- moved IRQ_conn1 217.2 mm to (-19.7, 76.2)
- moved INTERNAL_DATA_CONN2 187.8 mm to (27.0, 57.2)
- moved U76 169.3 mm to (154.0, 204.6)
- moved U82 163.9 mm to (57.3, 24.3)
- moved ML5 157.9 mm to (154.0, 177.6)
- moved IntBoardConn2 153.2 mm to (314.0, 43.2)
- moved U85 146.6 mm to (315.2, 24.3)
- moved U72 146.4 mm to (154.0, 150.6)
- moved CONN_DATA3 138.2 mm to (165.5, 177.8)
- moved U86 134.9 mm to (326.1, 24.3)
- moved ALU_DATA_BUS1 134.4 mm to (170.2, 177.8)
- moved U90 133.0 mm to (293.5, 24.3)
- moved AROM_LOW1 132.2 mm to (113.8, 150.6)
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Connections:
- net SELa renamed SELa_PGdis
- net dbg_mcode0 renamed mcode0
- net dbg_mcode1 renamed mcode1
- net dbg_mcode10 renamed Net-(U11-Pad17)
- net dbg_mcode11 renamed Net-(U11-Pad16)
- net dbg_mcode13 renamed Net-(U11-Pad14)
- net dbg_mcode15 renamed Net-(U11-Pad12)
- net dbg_mcode2 renamed Net-(U10-Pad17)
- net dbg_mcode3 renamed Net-(U10-Pad16)
- net dbg_mcode4 renamed Net-(U10-Pad15)
- net dbg_mcode5 renamed Net-(U10-Pad14)
- net dbg_mcode6 renamed Net-(U10-Pad13)
- net dbg_mcode7 renamed /seq_reset_rq
- net dbg_mcode8 renamed Net-(U11-Pad19)
- net dbg_mcode9 renamed Net-(U11-Pad18)
- CONN_ADDRESS1 pad 1: Net-(CONN_ADDRESS1-Pad1) -> ADDR0
- CONN_ADDRESS1 pad 10: Net-(CONN_ADDRESS1-Pad10) -> ADDR9
- CONN_ADDRESS1 pad 11: Net-(CONN_ADDRESS1-Pad11) -> ADDR10
- CONN_ADDRESS1 pad 12: Net-(CONN_ADDRESS1-Pad12) -> ADDR11
- CONN_ADDRESS1 pad 13: Net-(CONN_ADDRESS1-Pad13) -> ADDR12
- CONN_ADDRESS1 pad 14: Net-(CONN_ADDRESS1-Pad14) -> ADDR13
- CONN_ADDRESS1 pad 15: Net-(CONN_ADDRESS1-Pad15) -> ADDR14
- CONN_ADDRESS1 pad 16: Net-(CONN_ADDRESS1-Pad16) -> ADDR15
- CONN_ADDRESS1 pad 2: Net-(CONN_ADDRESS1-Pad2) -> ADDR1
- CONN_ADDRESS1 pad 3: Net-(CONN_ADDRESS1-Pad3) -> ADDR2
- CONN_ADDRESS1 pad 4: Net-(CONN_ADDRESS1-Pad4) -> ADDR3
- CONN_ADDRESS1 pad 5: Net-(CONN_ADDRESS1-Pad5) -> ADDR4
- CONN_ADDRESS1 pad 6: Net-(CONN_ADDRESS1-Pad6) -> ADDR5
- CONN_ADDRESS1 pad 7: Net-(CONN_ADDRESS1-Pad7) -> ADDR6
- CONN_ADDRESS1 pad 8: Net-(CONN_ADDRESS1-Pad8) -> ADDR7
- CONN_ADDRESS1 pad 9: Net-(CONN_ADDRESS1-Pad9) -> ADDR8
- IRQ_conn1 pad 2: unconnected-(IRQ_conn1-Pad2) -> SAMPLE_IRQ
- ML7 pad 11: CLOCK -> SAMPLE_IRQ
- U24 pad 12: /seq_reset -> SAMPLE_IRQ
- U35 pad 11: Net-(CONN_ADDRESS1-Pad8) -> ADDR7
- U35 pad 12: Net-(CONN_ADDRESS1-Pad7) -> ADDR6
- U35 pad 13: Net-(CONN_ADDRESS1-Pad6) -> ADDR5
- U35 pad 14: Net-(CONN_ADDRESS1-Pad5) -> ADDR4
- U35 pad 15: Net-(CONN_ADDRESS1-Pad4) -> ADDR3
- U35 pad 16: Net-(CONN_ADDRESS1-Pad3) -> ADDR2
- U35 pad 17: Net-(CONN_ADDRESS1-Pad2) -> ADDR1
- U35 pad 18: Net-(CONN_ADDRESS1-Pad1) -> ADDR0
- U36 pad 11: Net-(CONN_ADDRESS1-Pad8) -> ADDR7
- U36 pad 12: Net-(CONN_ADDRESS1-Pad7) -> ADDR6
- U36 pad 13: Net-(CONN_ADDRESS1-Pad6) -> ADDR5
- U36 pad 14: Net-(CONN_ADDRESS1-Pad5) -> ADDR4
- U36 pad 15: Net-(CONN_ADDRESS1-Pad4) -> ADDR3
- U36 pad 16: Net-(CONN_ADDRESS1-Pad3) -> ADDR2
- U36 pad 17: Net-(CONN_ADDRESS1-Pad2) -> ADDR1
- U36 pad 18: Net-(CONN_ADDRESS1-Pad1) -> ADDR0
- U4 pad 13: /seq_reset -> SAMPLE_IRQ
- U42 pad 11: Net-(CONN_ADDRESS1-Pad16) -> ADDR15
- U42 pad 12: Net-(CONN_ADDRESS1-Pad15) -> ADDR14
- U42 pad 13: Net-(CONN_ADDRESS1-Pad14) -> ADDR13
- U42 pad 14: Net-(CONN_ADDRESS1-Pad13) -> ADDR12
- U42 pad 15: Net-(CONN_ADDRESS1-Pad12) -> ADDR11
- U42 pad 16: Net-(CONN_ADDRESS1-Pad11) -> ADDR10
- U42 pad 17: Net-(CONN_ADDRESS1-Pad10) -> ADDR9
- U42 pad 18: Net-(CONN_ADDRESS1-Pad9) -> ADDR8
- U7 pad 6: /seq_reset -> SAMPLE_IRQ
- U76 pad 8: Net-(U75-Pad3) -> Net-(U76-Pad8)
- U79 pad 12: unconnected-(U79-Pad12) -> Net-(U79-Pad12)
- U79 pad 13: unconnected-(U79-Pad13) -> IR0
- U80 pad 1: unconnected-(U80-Pad1) -> Net-(U76-Pad8)
- U80 pad 2: unconnected-(U80-Pad2) -> Net-(U80-Pad2)
- U80 pad 3: unconnected-(U80-Pad3) -> Net-(U75-Pad3)
