File: schematics/cpu5/cpu5.kicad_pcb (KiCad board)
At the start: 2 copper layers, 166 parts, among them J1 Conn_01x12, J2 Conn_01x03, J3 Conn_01x40, J4 Conn_01x05, J5 Conn_01x03, U1 74LS161, U10 74LS574, U100 CY62256-70PC, U101 74LS04, U102 74LS02, U103 74LS541, U104 74LS541, U105 74LS541, U106 74LS541, U107 74LS541, U108 74LS02, U109 74LS32, U11 74LS574, U110 AT28C64-20PI, U111 AT28C64-20PI, U112 74LS32, U113 74LS32, U114 74LS138, U115 74LS541, U116 74LS541, U117 74LS138, U118 74LS541, U119 74LS541, U12 74LS08, U13 74LS138, U14 74LS138, U15 74LS138, U16 74LS138, U17 74LS138, U18 74LS138, U19 74LS138, U2 74LS161, U20 74LS138, U21 74LS08, U22 74LS04, U23 74LS86, U24 74LS32, U25 74LS86, U26 74LS08, U27 74LS138, U28 74LS04, U29 74LS32, U3 74LS193, U30 74LS32, U31 74LS08, U32 74LS32, U33 74LS32, U34 74LS74, U35 74LS541, U36 74LS541, U37 74LS193, U38 74LS541, U39 74LS193, U4 74LS04, U40 74LS193, U41 74LS541, U42 74LS541, U43 74LS541, U44 74LS541, U45 74LS193, U46 74LS193, U47 74LS541, U48 74LS193, U49 74LS193, U5 74LS08, U50 74LS193, U51 74LS193, U52 74LS541, U53 74LS541, U54 74LS541, U55 74LS541, U56 74LS193, U57 74LS193, U58 74LS541, U59 74LS541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

Commit message: cmake pipeline
Parts:
- removed CONN_DATA1: Conn_01x08, Connector_PinHeader_2.54mm:PinHeader_1x08_P2.54mm_Vertical
- removed Jdbg1: Conn_01x12, Connector_PinHeader_2.54mm:PinHeader_1x12_P2.54mm_Vertical
- added IR_BUF1: 74LS574, Package_DIP:DIP-20_W7.62mm, F.Cu at (-186.2, -174.8)
- added IR_BUF2: 74LS574, Package_DIP:DIP-20_W7.62mm, F.Cu at (-175.3, -174.8)
- added IR_BUF3: 74LS574, Package_DIP:DIP-20_W7.62mm, F.Cu at (-215.2, -75.5)
- added ML10: 74LS574, Package_DIP:DIP-20_W7.62mm, F.Cu at (58.9, -201.8)
- added ML11: 74LS574, Package_DIP:DIP-20_W7.62mm, F.Cu at (48.0, -201.8)
- added ML9: 74LS574, Package_DIP:DIP-20_W7.62mm, F.Cu at (37.2, -174.8)
- added U120: AS6C4008-55PCN, Package_DIP:DIP-32_W15.24mm, F.Cu at (-47.7, -159.0)
- added U121: 74LS32, Package_DIP:DIP-14_W7.62mm, F.Cu at (69.7, -162.9)
- added U122: 74LS541, Package_DIP:DIP-20_W7.62mm, F.Cu at (-142.8, -201.8)
- added U123: 74LS08, Package_DIP:DIP-14_W7.62mm, F.Cu at (35.8, -147.8)
- added U124: 74LS32, Package_DIP:DIP-14_W7.62mm, F.Cu at (-110.2, -162.9)
- added U125: 74LS32, Package_DIP:DIP-14_W7.62mm, F.Cu at (-157.9, -133.4)
- added U126: 74LS04, Package_DIP:DIP-14_W7.62mm, F.Cu at (-147.0, -133.4)
- added U127: 74LS08, Package_DIP:DIP-14_W7.62mm, F.Cu at (141.3, -201.8)
- added U128: 74LS74, Package_DIP:DIP-14_W7.62mm, F.Cu at (152.1, -201.8)
- added U129: 74LS74, Package_DIP:DIP-14_W7.62mm, F.Cu at (104.1, -159.9)
- added U130: 74LS04, Package_DIP:DIP-14_W7.62mm, F.Cu at (114.9, -182.3)
- added U131: 74LS74, Package_DIP:DIP-14_W7.62mm, F.Cu at (58.9, -174.8)
- added U132: 74LS541, Package_DIP:DIP-20_W7.62mm, F.Cu at (-216.8, -164.6)
- added U133: 74LS32, Package_DIP:DIP-14_W7.62mm, F.Cu at (-121.1, -179.8)
- added U134: 74LS32, Package_DIP:DIP-14_W7.62mm, F.Cu at (-131.9, -141.1)
- added U135: 74LS08, Package_DIP:DIP-14_W7.62mm, F.Cu at (-110.2, -201.8)
- added U136: 74LS541, Package_DIP:DIP-20_W7.62mm, F.Cu at (-209.0, -21.5)
- moved U82 341.9 mm to (-227.6, -164.6)
- moved U63 340.3 mm to (-209.0, -48.5)
- moved IR1 340.3 mm to (-186.2, -201.8)
- moved U26 337.4 mm to (-77.7, -201.8)
- moved U53 336.6 mm to (-230.7, -21.5)
- moved U100 333.4 mm to (-43.1, -201.8)
- moved U4 332.9 mm to (-182.7, -109.0)
- moved DbgConn2 330.1 mm to (-232.2, -159.6)
- moved U94 330.0 mm to (26.3, -201.8)
- moved U34 330.0 mm to (-204.4, -115.7)
- moved U10 329.5 mm to (-175.3, -201.8)
- moved U36 329.5 mm to (-164.5, -201.8)
- moved U29 328.9 mm to (-164.5, -152.8)
- moved U113 327.1 mm to (69.7, -201.8)
- moved U18 326.9 mm to (-121.1, -201.8)
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Connections:
- net Net-(U10-Pad13) renamed mcode6
- net Net-(U10-Pad14) renamed mcode5
- net Net-(U10-Pad15) renamed mcode4
- net Net-(U10-Pad16) renamed mcode3
- net Net-(U10-Pad17) renamed mcode2
- IR1 pad 2: iIR0 -> preIR0
- IR1 pad 3: iIR1 -> preIR1
- IR1 pad 4: iIR2 -> preIR2
- IR1 pad 5: iIR3 -> preIR3
- IR1 pad 6: iIR4 -> preIR4
- IR1 pad 7: iIR5 -> preIR5
- IR1 pad 8: iIR6 -> preIR6
- IR1 pad 9: iIR7 -> preIR7
- IntBoardConn2 pad 2: INT1 -> MMU_FAULT
- J1 pad 9: cword_en -> cword_clk
- ML7 pad 2: Net-(ML7-Pad2) -> FAULT_PENDING
- ML7 pad 3: DBG_PRE_INT1 -> Net-(ML7-Pad3)
- ML7 pad 4: DBG_PRE_INT2 -> Net-(ML7-Pad4)
- ML7 pad 5: DBG_PRE_INT3 -> Net-(ML7-Pad5)
- ML8 pad 1: PGE_bar -> GND
- U1 pad 3: GND -> Net-(IR_BUF2-Pad15)
- U1 pad 4: GND -> Net-(IR_BUF2-Pad14)
- U1 pad 5: GND -> Net-(IR_BUF2-Pad13)
- U1 pad 6: GND -> Net-(IR_BUF2-Pad12)
- U10 pad 11: cword_en -> cword_clk
- U10 pad 12: /seq_reset_rq -> mcode7
- U100 pad 22: MREAD -> MREAD_f
- U100 pad 27: MWRITE -> MWRITE_f
- U101 pad 5: unconnected-(U101-Pad5) -> Net-(U101-Pad5)
- U101 pad 6: unconnected-(U101-Pad6) -> EXTRAM_SEL
- U102 pad 10: PGE_bar -> Net-(U102-Pad10)
- U102 pad 4: PGE -> Net-(U102-Pad4)
- U102 pad 6: PGE_bar -> Net-(U102-Pad10)
- U102 pad 8: PGE -> Net-(U102-Pad4)
- U108 pad 11: unconnected-(U108-Pad11) -> TLBFD0
- U108 pad 12: unconnected-(U108-Pad12) -> MREAD
- U108 pad 13: unconnected-(U108-Pad13) -> Net-(U108-Pad13)
- U108 pad 4: unconnected-(U108-Pad4) -> Net-(U108-Pad4)
- U108 pad 5: unconnected-(U108-Pad5) -> TLBFD1
- U108 pad 6: unconnected-(U108-Pad6) -> MWRITE
- U11 pad 11: cword_en -> cword_clk
- U11 pad 12: Net-(U11-Pad12) -> LOAD_FAULT
- U113 pad 10: unconnected-(U113-Pad10) -> is_write_fault
- U113 pad 11: unconnected-(U113-Pad11) -> MWRITE_f
- U113 pad 12: unconnected-(U113-Pad12) -> MWRITE
- U113 pad 13: unconnected-(U113-Pad13) -> is_write_fault
- U113 pad 8: unconnected-(U113-Pad8) -> MMU_FAULT
- U113 pad 9: unconnected-(U113-Pad9) -> is_read_fault
- U117 pad 10: unconnected-(U117-Pad10) -> RD_FLT_0
- U117 pad 7: unconnected-(U117-Pad7) -> RD_FLT_2
- U117 pad 9: unconnected-(U117-Pad9) -> RD_FLT_1
- U13 pad 5: Net-(U11-Pad12) -> GND
- U14 pad 5: Net-(U11-Pad12) -> GND
- U15 pad 5: Net-(U11-Pad12) -> GND
- U16 pad 5: Net-(U11-Pad12) -> GND
- U17 pad 5: Net-(U17-Pad5) -> GND
- U18 pad 5: Net-(U17-Pad5) -> GND
- U19 pad 5: Net-(U17-Pad5) -> GND
- U2 pad 11: Net-(Jdbg1-Pad6) -> Net-(U124-Pad10)
- U2 pad 12: Net-(Jdbg1-Pad5) -> Net-(U124-Pad9)
- U2 pad 13: Net-(Jdbg1-Pad4) -> Net-(U124-Pad5)
- U2 pad 14: Net-(Jdbg1-Pad3) -> Net-(U124-Pad4)
- U2 pad 3: GND -> Net-(IR_BUF2-Pad19)
- U2 pad 4: GND -> Net-(IR_BUF2-Pad18)
- U2 pad 5: GND -> Net-(IR_BUF2-Pad17)
- U2 pad 6: GND -> Net-(IR_BUF2-Pad16)
- U20 pad 5: Net-(U17-Pad5) -> GND
- U24 pad 12: SAMPLE_IRQ -> /seq_reset
- U31 pad 9: unconnected-(U31-Pad9) -> IRQ
- U32 pad 10: init_ir -> IRi
- U32 pad 9: IRi -> start_instr
- U4 pad 1: unconnected-(U4-Pad1) -> Net-(U125-Pad8)
- U4 pad 2: unconnected-(U4-Pad2) -> Net-(U4-Pad2)
- U4 pad 3: Net-(U4-Pad3) -> Net-(U124-Pad11)
- U4 pad 4: Net-(U4-Pad4) -> start_phase
- U4 pad 8: Net-(U17-Pad5) -> LOAD_FAULT_bar
- U4 pad 9: Net-(U11-Pad12) -> LOAD_FAULT
- U5 pad 1: Net-(Jdbg1-Pad3) -> Net-(U4-Pad2)
- U5 pad 10: Net-(Jdbg1-Pad5) -> Net-(U5-Pad10)
- U5 pad 2: Net-(Jdbg1-Pad4) -> Net-(U124-Pad9)
- U5 pad 3: Net-(Jdbg1-Pad1) -> cword_clk
- U5 pad 4: Net-(Jdbg1-Pad5) -> Net-(U124-Pad4)
- U5 pad 5: Net-(Jdbg1-Pad6) -> Net-(U124-Pad5)
- U5 pad 6: Net-(Jdbg1-Pad2) -> Net-(U5-Pad10)
- U5 pad 8: cword_en -> end_phase
- U5 pad 9: Net-(Jdbg1-Pad3) -> phase_write
- U62 pad 2: DATA0 -> Net-(IR_BUF3-Pad19)
- U62 pad 3: DATA1 -> Net-(IR_BUF3-Pad18)
- U62 pad 4: DATA2 -> Net-(IR_BUF3-Pad17)
- U62 pad 5: DATA3 -> Net-(IR_BUF3-Pad16)
- U62 pad 6: DATA4 -> Net-(IR_BUF3-Pad15)
- U62 pad 7: DATA5 -> Net-(IR_BUF3-Pad14)
- U62 pad 8: DATA6 -> Net-(IR_BUF3-Pad13)
- U62 pad 9: DATA7 -> Net-(IR_BUF3-Pad12)
- U7 pad 1: Net-(U4-Pad4) -> end_phase
- U7 pad 10: Net-(Jdbg1-Pad2) -> start_phase
- U7 pad 11: phase_mread -> Net-(U135-Pad12)
- U7 pad 12: Net-(Jdbg1-Pad6) -> Net-(U126-Pad10)
- U7 pad 13: Net-(U4-Pad4) -> start_phase
- U7 pad 2: Net-(Jdbg1-Pad2) -> mcode7
- U7 pad 3: phase_write -> /seq_reset
- U7 pad 4: Net-(U4-Pad3) -> Net-(U124-Pad9)
- U7 pad 5: /seq_reset_rq -> Net-(U124-Pad10)
- U7 pad 6: SAMPLE_IRQ -> phase_write
- U7 pad 8: Net-(U4-Pad3) -> start_instr
- U7 pad 9: Net-(Jdbg1-Pad1) -> Net-(U126-Pad12)
- U8 pad 11: iIR3 -> Net-(U133-Pad12)
- U8 pad 3: iIR0 -> Net-(U133-Pad1)
- U8 pad 6: iIR1 -> Net-(U133-Pad4)
- U8 pad 8: iIR2 -> Net-(U133-Pad9)
- U83 pad 2: Net-(U83-Pad2) -> DBG_PRE_INT1
- U83 pad 3: DBG_PRE_INT1 -> Net-(ML7-Pad3)
- U84 pad 10: Net-(U83-Pad2) -> DBG_PRE_INT1
- U84 pad 13: Net-(U84-Pad13) -> DBG_PRE_INT2
- U84 pad 3: Net-(U84-Pad3) -> Net-(U130-Pad1)
- U84 pad 6: Net-(U84-Pad6) -> Net-(U130-Pad5)
- U84 pad 9: Net-(ML7-Pad2) -> FAULT_PENDING
- U85 pad 3: Net-(U85-Pad3) -> Net-(U130-Pad3)
- U86 pad 3: Net-(ML7-Pad2) -> FAULT_PENDING
- U87 pad 1: Net-(ML7-Pad2) -> unconnected-(U87-Pad1)
- U87 pad 10: Net-(U83-Pad2) -> unconnected-(U87-Pad10)
- U87 pad 11: Net-(U83-Pad2) -> unconnected-(U87-Pad11)
- U87 pad 12: INT1 -> unconnected-(U87-Pad12)
- U87 pad 13: Net-(U87-Pad13) -> unconnected-(U87-Pad13)
- U87 pad 2: Net-(U84-Pad3) -> unconnected-(U87-Pad2)
- U87 pad 3: Net-(U87-Pad3) -> unconnected-(U87-Pad3)
- U87 pad 4: Net-(U87-Pad3) -> unconnected-(U87-Pad4)
- U87 pad 5: Net-(ML7-Pad2) -> unconnected-(U87-Pad5)
- U87 pad 6: INT0 -> unconnected-(U87-Pad6)
- U87 pad 8: Net-(U85-Pad3) -> unconnected-(U87-Pad8)
- U87 pad 9: Net-(U87-Pad13) -> unconnected-(U87-Pad9)
- U88 pad 1: Net-(U84-Pad13) -> unconnected-(U88-Pad1)
- U88 pad 2: Net-(U84-Pad6) -> unconnected-(U88-Pad2)
- U88 pad 3: Net-(U88-Pad3) -> unconnected-(U88-Pad3)
- U88 pad 4: Net-(U88-Pad3) -> unconnected-(U88-Pad4)
- U88 pad 5: Net-(U84-Pad13) -> unconnected-(U88-Pad5)
- U88 pad 6: INT2 -> unconnected-(U88-Pad6)
- U89 pad 5: Net-(U84-Pad13) -> DBG_PRE_INT2
- U89 pad 6: DBG_PRE_INT2 -> Net-(ML7-Pad4)
- U89 pad 8: DBG_PRE_INT3 -> Net-(ML7-Pad5)
- U9 pad 11: iIR7 -> Net-(U134-Pad12)
- U9 pad 3: iIR4 -> Net-(U134-Pad1)
- U9 pad 6: iIR5 -> Net-(U134-Pad4)
- U9 pad 8: iIR6 -> Net-(U134-Pad9)
- U92 pad 11: unconnected-(U92-Pad11) -> FAULT
- U92 pad 12: unconnected-(U92-Pad12) -> MMU_FAULT
- U92 pad 13: unconnected-(U92-Pad13) -> GND
- U95 pad 13: Net-(U95-Pad13) -> Net-(U101-Pad5)
- U95 pad 8: Net-(U95-Pad13) -> Net-(U101-Pad5)
- U96 pad 5: Net-(U95-Pad13) -> Net-(U101-Pad5)
- U98 pad 22: MREAD -> MREAD_f
- U99 pad 11: unconnected-(U99-Pad11) -> Net-(U123-Pad10)
- U99 pad 12: unconnected-(U99-Pad12) -> Net-(U108-Pad4)
- U99 pad 13: unconnected-(U99-Pad13) -> PGE
