File: schematics/cpu5/memory.kicad_sch (KiCad schematic)
At the start: 37 parts, among them U100 CY62256-70PC, U101 74LS04, U102 74LS02, U103 74LS541, U104 74LS541, U105 74LS541, U106 74LS541, U107 74LS541, U108 74LS02, U109 74LS32, U110 AT28C64-20PI, U111 AT28C64-20PI, U112 74LS32, U113 74LS32, U114 74LS138, U115 74LS541, U116 74LS541, U117 74LS138, U118 74LS541, U119 74LS541, U120 AS6C4008-55PCN, U121 74LS32, U123 74LS08, U131 74LS74, U94 74LS541, U95 74LS32, U96 74LS138, U97 74LS00, U98 28C256, U99 74LS08

Commit message: faults fixed
Connections:
- net +5V: now also U131.10 (nS2)
- net MMU_FAULT: now also U131.9 (Q2); no longer U113.8 (Y3)
- net RESET: now also U131.13 (nR2)
- net CLOCK: now reaches U101.3 (A1)
- net at U101.4 (Y1): now also U131.11 (Clk2)
- net at U131.12 (D2): now also U113.8 (Y3)
Other:
- moved on the sheet: U101B, U131B
Changed lines of the file:
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@@
     (stroke (width 0) (type default) (color 0 0 0 0))
   )
+  (wire (pts (xy 561.34 203.2) (xy 617.22 203.2))
+    (stroke (width 0) (type default) (color 0 0 0 0))
+  )
   (wire (pts (xy 265.43 347.98) (xy 265.43 349.25))
     (stroke (width 0) (type default) (color 0 0 0 0))
@@
     (stroke (width 0) (type default) (color 0 0 0 0))
   )
+  (wire (pts (xy 632.46 203.2) (xy 635 203.2))
+    (stroke (width 0) (type default) (color 0 0 0 0))
+  )
   (wire (pts (xy 139.7 325.12) (xy 140.97 325.12))
     (stroke (width 0) (type default) (color 0 0 0 0))
@@
     (stroke (width 0) (type default) (color 0 0 0 0))
   )
+  (wire (pts (xy 614.68 205.74) (xy 617.22 205.74))
+    (stroke (width 0) (type default) (color 0 0 0 0))
+  )
   (wire (pts (xy 232.41 163.83) (xy 234.95 163.83))
     (stroke (width 0) (type default) (color 0 0 0 0))
@@
     (stroke (width 0) (type default) (color 0 0 0 0))
   )
-  (wire (pts (xy 561.34 203.2) (xy 607.06 203.2))
-    (stroke (width 0) (type default) (color 0 0 0 0))
-  )
   (wire (pts (xy 543.56 297.18) (xy 544.83 297.18))
     (stroke (width 0) (type default) (color 0 0 0 0))
@@
     (stroke (width 0) (type default) (color 0 0 0 0))
   )
+  (wire (pts (xy 614.68 226.06) (xy 614.68 205.74))
+    (stroke (width 0) (type default) (color 0 0 0 0))
+  )
   (wire (pts (xy 570.23 30.48) (xy 572.77 30.48))
     (stroke (width 0) (type default) (color 0 0 0 0))
@@
     (stroke (width 0) (type default) (color 0 0 0 0))
   )
+  (wire (pts (xy 624.84 194.31) (xy 624.84 198.12))
+    (stroke (width 0) (type default) (color 0 0 0 0))
+  )
   (wire (pts (xy 134.62 227.33) (xy 140.97 227.33))
     (stroke (width 0) (type default) (color 0 0 0 0))
@@
     (stroke (width 0) (type default) (color 0 0 0 0))
   )
+  (wire (pts (xy 607.06 226.06) (xy 614.68 226.06))
+    (stroke (width 0) (type default) (color 0 0 0 0))
+  )
   (wire (pts (xy 336.55 240.03) (xy 336.55 241.3))
     (stroke (width 0) (type default) (color 0 0 0 0))
@@
     (stroke (width 0) (type default) (color 0 0 0 0))
   )
+  (wire (pts (xy 624.84 213.36) (xy 624.84 215.9))
+    (stroke (width 0) (type default) (color 0 0 0 0))
+  )
   (wire (pts (xy 367.03 364.49) (xy 367.03 372.11))
     (stroke (width 0) (type default) (color 0 0 0 0))
@@
     (stroke (width 0) (type default) (color 0 0 0 0))
   )
+  (wire (pts (xy 588.01 226.06) (xy 591.82 226.06))
+    (stroke (width 0) (type default) (color 0 0 0 0))
+  )
   (wire (pts (xy 228.6 187.96) (xy 229.87 187.96))
     (stroke (width 0) (type default) (color 0 0 0 0))
@@
     (stroke (width 0) (type default) (color 0 0 0 0))
   )
+  (wire (pts (xy 624.84 215.9) (xy 626.11 215.9))
+    (stroke (width 0) (type default) (color 0 0 0 0))
+  )
   (wire (pts (xy 382.27 77.47) (xy 383.54 77.47))
     (stroke (width 0) (type default) (color 0 0 0 0))
@@
     )
   )
+  (global_label "RESET" (shape input) (at 626.11 215.9 0) (fields_autoplaced)
+    (effects (font (size 1.27 1.27)) (justify left))
+    (property "Intersheet References" "${INTERSHEET_REFS}" (id 0) (at 634.2683 215.8206 0)
+      (effects (font (size 1.27 1.27)) (justify left) hide)
+    )
+  )
   (global_label "READ_TLB" (shape input) (at 289.56 313.69 0) (fields_autoplaced)
     (effects (font (size 1.27 1.27)) (justify left))
@@
     )
   )
+  (global_label "CLOCK" (shape input) (at 588.01 226.06 180) (fields_autoplaced)
+    (effects (font (size 1.27 1.27)) (justify right))
+    (property "Intersheet References" "${INTERSHEET_REFS}" (id 0) (at 579.4283 225.9806 0)
+      (effects (font (size 1.27 1.27)) (justify right) hide)
+    )
+  )
   (global_label "TLBA11" (shape input) (at 266.7 361.95 0) (fields_autoplaced)
     (effects (font (size 1.27 1.27)) (justify left))
@@
     )
   )
-  (global_label "MMU_FAULT" (shape input) (at 607.06 203.2 0) (fields_autoplaced)
+  (global_label "MMU_FAULT" (shape input) (at 635 203.2 0) (fields_autoplaced)
     (effects (font (size 1.27 1.27)) (justify left))
-    (property "Intersheet References" "${INTERSHEET_REFS}" (id 0) (at 620.1774 203.1206 0)
+    (property "Intersheet References" "${INTERSHEET_REFS}" (id 0) (at 648.1174 203.1206 0)
       (effects (font (size 1.27 1.27)) (justify left) hide)
     )
@@
     (pin "9")
   )
-  (symbol (lib_id "7400_ice:74LS04") (at 596.9 128.27 0) (unit 2)
+  (symbol (lib_id "7400_ice:74LS04") (at 599.44 226.06 0) (unit 2)
     (in_bom yes) (on_board yes) (fields_autoplaced)
-    (property "Reference" "U101" (id 0) (at 596.9 114.3 0))
-    (property "Value" "74LS04" (id 1) (at 596.9 116.84 0))
-    (property "Footprint" "Package_DIP:DIP-14_W7.62mm" (id 2) (at 596.9 128.27 0)
+    (property "Reference" "U101" (id 0) (at 599.44 212.09 0))
+    (property "Value" "74LS04" (id 1) (at 599.44 214.63 0))
+    (property "Footprint" "Package_DIP:DIP-14_W7.62mm" (id 2) (at 599.44 226.06 0)
       (effects (font (size 1.27 1.27)) hide)
     )
-    (property "Datasheet" "http://www.ti.com/lit/gpn/sn74LS04" (id 3) (at 595.63 133.35 0)
+    (property "Datasheet" "http://www.ti.com/lit/gpn/sn74LS04" (id 3) (at 598.17 231.14 0)
       (effects (font (size 1.27 1.27)) hide)
     )
-    (property "VerilogInclude" "icechips/7404.v" (id 4) (at 596.9 119.38 0))
-    (property "VerilogCode" "ttl_7404 core (.A(`A), .Y(`Y));" (id 5) (at 596.9 121.92 0))
+    (property "VerilogInclude" "icechips/7404.v" (id 4) (at 599.44 217.17 0))
+    (property "VerilogCode" "ttl_7404 core (.A(`A), .Y(`Y));" (id 5) (at 599.44 219.71 0))
     (pin "3")
     (pin "4")
@@
     (pin "1")
   )
-  (symbol (lib_id "7400_ice:74LS74") (at 265.43 34.29 0) (unit 2)
+  (symbol (lib_id "7400_ice:74LS74") (at 624.84 205.74 0) (unit 2)
     (in_bom yes) (on_board yes) (fields_autoplaced)
-    (property "Reference" "U131" (id 0) (at 267.4494 24.13 0)
+    (property "Reference" "U131" (id 0) (at 626.8594 195.58 0)
       (effects (font (size 1.27 1.27)) (justify left))
     )
-    (property "Value" "74LS74" (id 1) (at 267.4494 26.67 0)
+    (property "Value" "74LS74" (id 1) (at 626.8594 198.12 0)
       (effects (font (size 1.27 1.27)) (justify left))
     )
-    (property "Footprint" "Package_DIP:DIP-14_W7.62mm" (id 2) (at 265.43 34.29 0)
+    (property "Footprint" "Package_DIP:DIP-14_W7.62mm" (id 2) (at 624.84 205.74 0)
       (effects (font (size 1.27 1.27)) hide)
     )
-    (property "Datasheet" "74xx/74hc_hct74.pdf" (id 3) (at 247.65 22.86 0)
+    (property "Datasheet" "74xx/74hc_hct74.pdf" (id 3) (at 607.06 194.31 0)
       (effects (font (size 1.27 1.27)) hide)
     )
-    (property "VerilogInclude" "icechips/7474.v" (id 4) (at 265.43 34.29 0)
+    (property "VerilogInclude" "icechips/7474.v" (id 4) (at 624.84 205.74 0)
       (effects (font (size 1.27 1.27)) hide)
     )
-    (property "VerilogCode" "ttl_7474 core (.Preset_bar({nS2, nS1}), .Clear_bar({nR2, nR1}), .D({D2,D1}), .Clk({Clk2,Clk1}), .Q({Q2,Q1}), .Q_bar({nQ2,nQ1}));" (id 5) (at 265.43 34.29 0)
+    (property "VerilogCode" "ttl_7474 core (.Preset_bar({nS2, nS1}), .Clear_bar({nR2, nR1}), .D({D2,D1}), .Clk({Clk2,Clk1}), .Q({Q2,Q1}), .Q_bar({nQ2,nQ1}));" (id 5) (at 624.84 205.74 0)
       (effects (font (size 1.27 1.27)) hide)
     )
@@
     (pin "3")
   )
+  (symbol (lib_id "power:+5V") (at 624.84 194.31 0) (unit 1)
+    (in_bom yes) (on_board yes) (fields_autoplaced)
+    (property "Reference" "#PWR?" (id 0) (at 624.84 198.12 0)
+      (effects (font (size 1.27 1.27)) hide)
+    )
+    (property "Value" "+5V" (id 1) (at 627.38 193.0399 0)
+      (effects (font (size 1.27 1.27)) (justify left))
+    )
+    (property "Footprint" "" (id 2) (at 624.84 194.31 0)
+      (effects (font (size 1.27 1.27)) hide)
+    )
+    (property "Datasheet" "" (id 3) (at 624.84 194.31 0)
+      (effects (font (size 1.27 1.27)) hide)
+    )
+    (pin "1")
+  )
   (symbol (lib_id "7400_ice:74LS541") (at 153.67 280.67 0) (unit 1)
